File: Fan_Control.kicad_sch (KiCad schematic)
At the start: 2 parts, among them J10 Conn_01x04, J9 Conn_01x04

Commit message: Second draft of placement and wiring.
Connections:
- net Fan_1_Control: now also J9.3 (Pin_3); no longer J9.2 (Pin_2)
- net Fan_1_PWM: now also J9.4 (Pin_4); no longer J9.3 (Pin_3)
- net Fan_1_Power: now also J9.2 (Pin_2); no longer J9.1 (Pin_1)
- net Fan_2_Control: now also J10.3 (Pin_3); no longer J10.2 (Pin_2)
- net Fan_2_PWM: now also J10.4 (Pin_4); no longer J10.3 (Pin_3)
- net Fan_2_Power: now also J10.2 (Pin_2); no longer J10.1 (Pin_1)
- net To_GND_1: now also J9.1 (Pin_1); no longer J9.4 (Pin_4)
- net To_GND_2: now also J10.1 (Pin_1); no longer J10.4 (Pin_4)
Changed lines of the file:
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@@
+		)
+	)
+	(hierarchical_label "To_GND_2"
+		(shape output)
+		(at 119.38 104.14 90)
+		(effects
+			(font
+				(size 1.27 1.27)
+			)
+			(justify left)
+		)
+	)
+	(hierarchical_label "To_GND_1"
+		(shape output)
+		(at 57.15 104.14 90)
+		(effects
+			(font
+				(size 1.27 1.27)
+			)
+			(justify left)
+		)
+	)
+	(hierarchical_label "Fan_2_PWM"
+		(shape input)
+		(at 142.24 124.46 270)
+		(effects
+			(font
+				(size 1.27 1.27)
+			)
+			(justify right)
+		)
+	)
+	(hierarchical_label "Fan_2_Control"
+		(shape input)
+		(at 137.16 113.03 180)
+		(effects
+			(font
+				(size 1.27 1.27)
+			)
+			(justify right)
 		)
 	)
 	(hierarchical_label "Fan_1_Control"
+		(shape input)
+		(at 77.47 113.03 180)
+		(effects
+			(font
+				(size 1.27 1.27)
+			)
+			(justify right)
+		)
+	)
+	(hierarchical_label "Fan_1_Power"
 		(shape input)
 		(at 77.47 110.49 180)
@@
 		)
 	)
-	(hierarchical_label "Fan_2_Control"
+	(hierarchical_label "Fan_2_Power"
 		(shape input)
 		(at 137.16 110.49 180)
@@
 	(hierarchical_label "Fan_1_PWM"
 		(shape input)
-		(at 77.47 113.03 180)
-		(effects
-			(font
-				(size 1.27 1.27)
-			)
-			(justify right)
-		)
-	)
-	(hierarchical_label "To_GND_2"
-		(shape output)
-		(at 142.24 124.46 270)
-		(effects
-			(font
-				(size 1.27 1.27)
-			)
-			(justify right)
-		)
-	)
-	(hierarchical_label "To_GND_1"
-		(shape output)
 		(at 81.28 124.46 270)
 		(effects
 			(font
-				(size 1.27 1.27)
-			)
-			(justify right)
-		)
-	)
-	(hierarchical_label "Fan_1_Power"
-		(shape input)
-		(at 57.15 104.14 180)
-		(effects
-			(font
-				(size 1.27 1.27)
-			)
-			(justify right)
-		)
-	)
-	(hierarchical_label "Fan_2_PWM"
-		(shape input)
-		(at 137.16 113.03 180)
-		(effects
-			(font
-				(size 1.27 1.27)
-			)
-			(justify right)
-		)
-	)
-	(hierarchical_label "Fan_2_Power"
-		(shape input)
-		(at 119.38 104.14 180)
-		(effects
-			(font
