File: gse_control_node.kicad_sch (KiCad schematic)
At the start: 8 parts, among them J1 Screw_Terminal_01x02

Commit message: add all lcsc part numbers
Parts:
- R1: LCSC (none) -> C137992
- R2, R3: LCSC (none) -> C106235
Changed lines of the file:
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@@
 			)
 		)
-		(property "LCSC" ""
+		(property "LCSC" "C106235"
 			(at 107.95 27.94 0)
 			(hide yes)
@@
 			)
 		)
-		(property "LCSC" ""
+		(property "LCSC" "C137992"
 			(at 77.47 24.13 0)
 			(hide yes)
@@
 			)
 		)
-		(property "LCSC" ""
-			(at 116.84 27.94 0)
-			(hide yes)
+		(property "LCSC" "C106235"
+			(at 116.84 27.94 0)
+			(hide yes)

Commit message: add a 12v testpoint
Parts:
- R1: LCSC C137992 -> (none)
- R2, R3: LCSC C106235 -> (none)
Changed lines of the file:
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@@
 			)
 		)
-		(property "LCSC" "C106235"
+		(property "LCSC" ""
 			(at 107.95 27.94 0)
 			(hide yes)
@@
 			)
 		)
-		(property "LCSC" "C137992"
+		(property "LCSC" ""
 			(at 77.47 24.13 0)
 			(hide yes)
@@
 			)
 		)
-		(property "LCSC" "C106235"
-			(at 116.84 27.94 0)
-			(hide yes)
+		(property "LCSC" ""
+			(at 116.84 27.94 0)
+			(hide yes)
