File: adc_filtering.kicad_sch (KiCad schematic)
At the start: 16 parts, among them U7 ADS112C04

Commit message: do some pcb routing
Parts:
- renumbered C24 to C1, C25 to C2, C26 to C3, C27 to C4, C28 to C5, C29 to C6, D6 to D1, D7 to D2, D8 to D3, D9 to D4, R21 to R4, R22 to R5, R23 to R6, R24 to R7, R25 to R8, U7 to U1
Changed lines of the file:
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@@
 		(dnp no)
 		(fields_autoplaced yes)
-		(property "Reference" "C25"
+		(property "Reference" "C2"
 			(at 119.38 134.6262 0)
 			(show_name no)
@@
 			(project "gse_control_node"
 				(path "/24817451-dfe0-4b9a-9d93-7304529c9d58/e6f03911-29ab-479a-bf6e-91fcd28c212a"
-					(reference "C25")
+					(reference "C2")
 					(unit 1)
 				)
@@
 		(in_pos_files yes)
 		(dnp no)
-		(property "Reference" "C26"
+		(property "Reference" "C3"
 			(at 132.08 50.292 90)
 			(show_name no)
@@
 			(project "gse_control_node"
 				(path "/24817451-dfe0-4b9a-9d93-7304529c9d58/e6f03911-29ab-479a-bf6e-91fcd28c212a"
-					(reference "C26")
+					(reference "C3")
 					(unit 1)
 				)
@@
 		(in_pos_files yes)
 		(dnp no)
-		(property "Reference" "#PWR0151"
+		(property "Reference" "#PWR010"
 			(at 105.41 146.05 0)
 			(hide yes)
@@
 			(project "gse_control_node"
 				(path "/24817451-dfe0-4b9a-9d93-7304529c9d58/e6f03911-29ab-479a-bf6e-91fcd28c212a"
-					(reference "#PWR0151")
+					(reference "#PWR010")
 					(unit 1)
 				)
@@
 		(dnp no)
 		(fields_autoplaced yes)
-		(property "Reference" "C24"
+		(property "Reference" "C1"
 			(at 107.95 134.6262 0)
 			(show_name no)
@@
 			(project "gse_control_node"
 				(path "/24817451-dfe0-4b9a-9d93-7304529c9d58/e6f03911-29ab-479a-bf6e-91fcd28c212a"
-					(reference "C24")
+					(reference "C1")
 					(unit 1)
 				)
@@
 		(in_pos_files yes)
 		(dnp no)
-		(property "Reference" "U7"
+		(property "Reference" "U1"
 			(at 145.796 139.7 0)
 			(show_name no)
@@
 			(project "gse_control_node"
 				(path "/24817451-dfe0-4b9a-9d93-7304529c9d58/e6f03911-29ab-479a-bf6e-91fcd28c212a"
-					(reference "U7")
+					(reference "U1")
 					(unit 1)
 				)
@@
 		(in_pos_files yes)
 		(dnp no)
-		(property "Reference" "D6"
+		(property "Reference" "D1"
 			(at 131.064 36.576 0)
 			(show_name no)
@@
 			(project "gse_control_node"
 				(path "/24817451-dfe0-4b9a-9d93-7304529c9d58/e6f03911-29ab-479a-bf6e-91fcd28c212a"
-					(reference "D6")
+					(reference "D1")
 					(unit 1)
 				)
@@
 		(in_pos_files yes)
 		(dnp no)
-		(property "Reference" "#PWR0158"
+		(property "Reference" "#PWR014"
 			(at 118.11 91.44 0)
 			(hide yes)
@@
 			(project "gse_control_node"
 				(path "/24817451-dfe0-4b9a-9d93-7304529c9d58/e6f03911-29ab-479a-bf6e-91fcd28c212a"
-					(reference "#PWR0158")
+					(reference "#PWR014")
 					(unit 1)
 				)
@@
 		(in_pos_files yes)
 		(dnp no)
-		(property "Reference" "C28"
+		(property "Reference" "C5"
 			(at 156.21 50.292 90)
 			(show_name no)
@@
 			(project "gse_control_node"
 				(path "/24817451-dfe0-4b9a-9d93-7304529c9d58/e6f03911-29ab-479a-bf6e-91fcd28c212a"
-					(reference "C28")
+					(reference "C5")
 					(unit 1)
 				)
@@
 		(in_pos_files yes)
 		(dnp no)
-		(property "Reference" "#PWR0159"
+		(property "Reference" "#PWR017"
 			(at 137.16 93.98 0)
 			(hide yes)
@@
 			(project "gse_control_node"
 				(path "/24817451-dfe0-4b9a-9d93-7304529c9d58/e6f03911-29ab-479a-bf6e-91fcd28c212a"
-					(reference "#PWR0159")
+					(reference "#PWR017")
 					(unit 1)
 				)
@@
 		(in_pos_files yes)
 		(dnp no)
-		(property "Reference" "#PWR0161"
+		(property "Reference" "#PWR013"
 			(at 118.11 44.45 0)
 			(hide yes)
@@
 			(project "gse_control_node"
 				(path "/24817451-dfe0-4b9a-9d93-7304529c9d58/e6f03911-29ab-479a-bf6e-91fcd28c212a"
-					(reference "#PWR0161")
+					(reference "#PWR013")
 					(unit 1)
 				)
@@
 		(in_pos_files yes)
 		(dnp no)
-		(property "Reference" "#PWR0153"
+		(property "Reference" "#PWR011"
 			(at 116.84 133.35 0)
 			(hide yes)
@@
 			(project "gse_control_node"
 				(path "/24817451-dfe0-4b9a-9d93-7304529c9d58/e6f03911-29ab-479a-bf6e-91fcd28c212a"
-					(reference "#PWR0153")
+					(reference "#PWR011")
 					(unit 1)
 				)
@@
 		(in_pos_files yes)
 		(dnp no)
-		(property "Reference" "R25"
+		(property "Reference" "R8"
 			(at 124.46 117.094 90)
 			(show_name no)
@@
 			(project "gse_control_node"
 				(path "/24817451-dfe0-4b9a-9d93-7304529c9d58/e6f03911-29ab-479a-bf6e-91fcd28c212a"
-					(reference "R25")
+					(reference "R8")
 					(unit 1)
 				)
@@
 		(in_pos_files yes)
 		(dnp no)
-		(property "Reference" "R23"
+		(property "Reference" "R6"
 			(at 115.062 66.294 90)
 			(show_name no)
@@
 			(project "gse_control_node"
 				(path "/24817451-dfe0-4b9a-9d93-7304529c9d58/e6f03911-29ab-479a-bf6e-91fcd28c212a"
-					(reference "R23")
+					(reference "R6")
 					(unit 1)
 				)
@@
 		(in_pos_files yes)
 		(dnp no)
-		(property "Reference" "R21"
+		(property "Reference" "R4"
 			(at 115.57 55.88 90)
 			(show_name no)
@@
 			(project "gse_control_node"
 				(path "/24817451-dfe0-4b9a-9d93-7304529c9d58/e6f03911-29ab-479a-bf6e-91fcd28c212a"
-					(reference "R21")
+					(reference "R4")
 					(unit 1)
 				)
@@
 		(in_pos_files yes)
 		(dnp no)
-		(property "Reference" "#PWR0152"
+		(property "Reference" "#PWR012"
 			(at 116.84 146.05 0)
 			(hide yes)
@@
 			(project "gse_control_node"
 				(path "/24817451-dfe0-4b9a-9d93-7304529c9d58/e6f03911-29ab-479a-bf6e-91fcd28c212a"
-					(reference "#PWR0152")
+					(reference "#PWR012")
 					(unit 1)
 				)
@@
 		(in_pos_files yes)
 		(dnp no)
-		(property "Reference" "#PWR0156"
+		(property "Reference" "#PWR020"
 			(at 161.29 46.99 0)
 			(hide yes)
@@
 			(project "gse_control_node"
 				(path "/24817451-dfe0-4b9a-9d93-7304529c9d58/e6f03911-29ab-479a-bf6e-91fcd28c212a"
-					(reference "#PWR0156")
+					(reference "#PWR020")
 					(unit 1)
 				)
@@
 		(in_pos_files yes)
 		(dnp no)
-		(property "Reference" "D9"
+		(property "Reference" "D4"
 			(at 156.21 91.948 0)
 			(show_name no)
@@
 			(project "gse_control_node"
 				(path "/24817451-dfe0-4b9a-9d93-7304529c9d58/e6f03911-29ab-479a-bf6e-91fcd28c212a"
-					(reference "D9")
+					(reference "D4")
 					(unit 1)
 				)
@@
 		(in_pos_files yes)
 		(dnp no)
-		(property "Reference" "R24"
+		(property "Reference" "R7"
 			(at 115.57 71.12 90)
 			(show_name no)
@@
 			(project "gse_control_node"
 				(path "/24817451-dfe0-4b9a-9d93-7304529c9d58/e6f03911-29ab-479a-bf6e-91fcd28c212a"
-					(reference "R24")
+					(reference "R7")
 					(unit 1)
 				)
@@
 		(in_pos_files yes)
 		(dnp no)
-		(property "Reference" "#PWR0150"
+		(property "Reference" "#PWR09"
 			(at 105.41 128.27 0)
 			(hide yes)
@@
 			(project "gse_control_node"
 				(path "/24817451-dfe0-4b9a-9d93-7304529c9d58/e6f03911-29ab-479a-bf6e-91fcd28c212a"
-					(reference "#PWR0150")
+					(reference "#PWR09")
 					(unit 1)
 				)
@@
 		(in_pos_files yes)
 		(dnp no)
-		(property "Reference" "#PWR0160"
+		(property "Reference" "#PWR019"
 			(at 142.24 91.44 0)
 			(hide yes)
@@
 			(project "gse_control_node"
 				(path "/24817451-dfe0-4b9a-9d93-7304529c9d58/e6f03911-29ab-479a-bf6e-91fcd28c212a"
-					(reference "#PWR0160")
+					(reference "#PWR019")
 					(unit 1)
 				)
@@
 		(in_pos_files yes)
 		(dnp no)
-		(property "Reference" "D8"
+		(property "Reference" "D3"
 			(at 155.194 36.576 0)
 			(show_name no)
@@
 			(project "gse_control_node"
 				(path "/24817451-dfe0-4b9a-9d93-7304529c9d58/e6f03911-29ab-479a-bf6e-91fcd28c212a"
-					(reference "D8")
+					(reference "D3")
 					(unit 1)
 				)
@@
 		(in_pos_files yes)
 		(dnp no)
-		(property "Reference" "#PWR0155"
+		(property "Reference" "#PWR018"
 			(at 142.24 44.45 0)
 			(hide yes)
@@
 			(project "gse_control_node"
 				(path "/24817451-dfe0-4b9a-9d93-7304529c9d58/e6f03911-29ab-479a-bf6e-91fcd28c212a"
-					(reference "#PWR0155")
+					(reference "#PWR018")
 					(unit 1)
 				)
@@
 		(in_pos_files yes)
 		(dnp no)
-		(property "Reference" "#PWR0157"
+		(property "Reference" "#PWR021"
 			(at 161.29 93.98 0)
 			(hide yes)
@@
 			(project "gse_control_node"
 				(path "/24817451-dfe0-4b9a-9d93-7304529c9d58/e6f03911-29ab-479a-bf6e-91fcd28c212a"
-					(reference "#PWR0157")
+					(reference "#PWR021")
 					(unit 1)
 				)
@@
 		(in_pos_files yes)
 		(dnp no)
-		(property "Reference" "C29"
+		(property "Reference" "C6"
 			(at 156.718 76.454 90)
 			(show_name no)
@@
 			(project "gse_control_node"
 				(path "/24817451-dfe0-4b9a-9d93-7304529c9d58/e6f03911-29ab-479a-bf6e-91fcd28c212a"
-					(reference "C29")
+					(reference "C6")
 					(unit 1)
 				)
@@
 		(in_pos_files yes)
 		(dnp no)
-		(property "Reference" "#PWR0149"
+		(property "Reference" "#PWR015"
 			(at 127 146.05 0)
 			(hide yes)
@@
 			(project "gse_control_node"
 				(path "/24817451-dfe0-4b9a-9d93-7304529c9d58/e6f03911-29ab-479a-bf6e-91fcd28c212a"
-					(reference "#PWR0149")
+					(reference "#PWR015")
 					(unit 1)
 				)
@@
 		(in_pos_files yes)
 		(dnp no)
-		(property "Reference" "D7"
+		(property "Reference" "D2"
 			(at 131.064 91.694 0)
 			(show_name no)
@@
 			(project "gse_control_node"
 				(path "/24817451-dfe0-4b9a-9d93-7304529c9d58/e6f03911-29ab-479a-bf6e-91fcd28c212a"
-					(reference "D7")
+					(reference "D2")
 					(unit 1)
 				)
@@
 		(in_pos_files yes)
 		(dnp no)
-		(property "Reference" "R22"
+		(property "Reference" "R5"
 			(at 115.062 61.214 90)
 			(show_name no)
@@
 			(project "gse_control_node"
 				(path "/24817451-dfe0-4b9a-9d93-7304529c9d58/e6f03911-29ab-479a-bf6e-91fcd28c212a"
-					(reference "R22")
+					(reference "R5")
 					(unit 1)
 				)
@@
 		(in_pos_files yes)
 		(dnp no)
-		(property "Reference" "C27"
+		(property "Reference" "C4"
 			(at 132.588 76.454 90)
 			(show_name no)
@@
 			(project "gse_control_node"
 				(path "/24817451-dfe0-4b9a-9d93-7304529c9d58/e6f03911-29ab-479a-bf6e-91fcd28c212a"
-					(reference "C27")
+					(reference "C4")
 					(unit 1)
 				)
@@
 		(in_pos_files yes)
 		(dnp no)
-		(property "Reference" "#PWR0154"
+		(property "Reference" "#PWR016"
 			(at 137.16 46.99 0)
 			(hide yes)
@@
 			(project "gse_control_node"
 				(path "/24817451-dfe0-4b9a-9d93-7304529c9d58/e6f03911-29ab-479a-bf6e-91fcd28c212a"
-					(reference "#PWR0154")
+					(reference "#PWR016")
 					(unit 1)
 				)

Commit message: remove unneccesary component fields
Parts:
- C1, C2: value 0.1μF -> 100nF; LCSC C307331 -> (none); MPN CL05B104KO5NNNC -> (none)
- C3, C4, C5, C6: LCSC C576725 -> (none)
- R4, R5, R6, R7: value 1k -> 1kΩ
- R8: value 10k -> 10kΩ; footprint Resistor_SMD:R_0402_1005Metric -> Resistor_SMD:R_0603_1608Metric; LCSC C25531 -> (none); MPN 0402WGJ0103TCE -> (none)
- U1: MPN ADS112C04IPWR -> (none)

Commit message: add all lcsc part numbers
Parts:
- C1, C2: LCSC (none) -> C85858
- C3, C4, C5, C6: value 150nF -> 220nF; LCSC (none) -> C77011
- R4, R5, R6, R7: value 1kΩ -> 680; LCSC (none) -> C137948
- R8: LCSC (none) -> C99198
Changed lines of the file:
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@@
 			)
 		)
-		(property "LCSC" ""
+		(property "LCSC" "C85858"
 			(at 116.84 135.89 0)
 			(hide yes)
@@
 			)
 		)
-		(property "Value" "150nF"
+		(property "Value" "220nF"
 			(at 133.35 52.324 90)
 			(show_name no)
@@
 			)
 		)
-		(property "LCSC" ""
+		(property "LCSC" "C77011"
 			(at 130.81 46.99 90)
 			(hide yes)
@@
 			)
 		)
-		(property "LCSC" ""
+		(property "LCSC" "C85858"
 			(at 105.41 135.89 0)
 			(hide yes)
@@
 			)
 		)
-		(property "Value" "150nF"
+		(property "Value" "220nF"
 			(at 157.48 52.324 90)
 			(show_name no)
@@
 			)
 		)
-		(property "LCSC" ""
+		(property "LCSC" "C77011"
 			(at 154.94 46.99 90)
 			(hide yes)
@@
 			)
 		)
-		(property "LCSC" ""
+		(property "LCSC" "C99198"
 			(at 124.46 121.92 0)
 			(hide yes)
@@
 			)
 		)
-		(property "Value" "1kΩ"
+		(property "Value" "680"
 			(at 119.634 66.294 90)
 			(show_name no)
@@
 			)
 		)
+		(property "LCSC" "C137948"
+			(at 119.38 68.58 90)
+			(hide yes)
+			(show_name no)
+			(do_not_autoplace no)
+			(effects
+				(font
+					(size 1.27 1.27)
+				)
+			)
+		)
 		(pin "2"
 		)
@@
 			)
 		)
-		(property "Value" "1kΩ"
+		(property "Value" "680"
 			(at 119.888 55.88 90)
 			(show_name no)
@@
 			)
 		)
+		(property "LCSC" "C137948"
+			(at 119.38 58.42 90)
+			(hide yes)
+			(show_name no)
+			(do_not_autoplace no)
+			(effects
+				(font
+					(size 1.27 1.27)
+				)
+			)
+		)
 		(pin "2"
 		)
@@
 			)
 		)
-		(property "Value" "1kΩ"
+		(property "Value" "680"
 			(at 119.888 71.12 90)
 			(show_name no)
@@
 		(property "Description" "Resistor, small US symbol"
 			(at 119.38 73.66 0)
+			(hide yes)
+			(show_name no)
+			(do_not_autoplace no)
+			(effects
+				(font
+					(size 1.27 1.27)
+				)
+			)
+		)
+		(property "LCSC" "C137948"
+			(at 119.38 73.66 90)
 			(hide yes)
 			(show_name no)
@@
 			)
 		)
-		(property "Value" "150nF"
+		(property "Value" "220nF"
 			(at 157.988 78.486 90)
 			(show_name no)
@@
 			)
 		)
-		(property "LCSC" ""
+		(property "LCSC" "C77011"
 			(at 154.94 81.28 90)
 			(hide yes)
@@
 			)
 		)
-		(property "Value" "1kΩ"
+		(property "Value" "680"
 			(at 119.634 61.214 90)
 			(show_name no)
@@
 			)
 		)
+		(property "LCSC" "C137948"
+			(at 119.38 63.5 90)
+			(hide yes)
+			(show_name no)
+			(do_not_autoplace no)
+			(effects
+				(font
+					(size 1.27 1.27)
+				)
+			)
+		)
 		(pin "2"
 		)
@@
 			)
 		)
-		(property "Value" "150nF"
+		(property "Value" "220nF"
 			(at 133.858 78.486 90)
 			(show_name no)
@@
 			)
 		)
-		(property "LCSC" ""
+		(property "LCSC" "C77011"
 			(at 130.81 81.28 90)
 			(hide yes)

Commit message: update all capacitors to jlcpcb basic components
Parts:
- C1, C2: LCSC C85858 -> C307331
- C3, C4, C5, C6: LCSC C77011 -> C16772
Changed lines of the file:
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@@
 			)
 		)
-		(property "LCSC" "C85858"
+		(property "LCSC" "C307331"
 			(at 116.84 135.89 0)
 			(hide yes)
@@
 			)
 		)
-		(property "LCSC" "C77011"
+		(property "LCSC" "C16772"
 			(at 130.81 46.99 90)
 			(hide yes)
@@
 			)
 		)
-		(property "LCSC" "C85858"
+		(property "LCSC" "C307331"
 			(at 105.41 135.89 0)
 			(hide yes)
@@
 			)
 		)
-		(property "LCSC" "C77011"
+		(property "LCSC" "C16772"
 			(at 154.94 46.99 90)
 			(hide yes)
@@
 			)
 		)
-		(property "LCSC" "C77011"
+		(property "LCSC" "C16772"
 			(at 154.94 81.28 90)
 			(hide yes)
@@
 			)
 		)
-		(property "LCSC" "C77011"
+		(property "LCSC" "C16772"
 			(at 130.81 81.28 90)
 			(hide yes)

Commit message: add a 12v testpoint
Parts:
- R4, R5, R6, R7: LCSC C137948 -> (none)
- R8: LCSC C99198 -> (none)
Changed lines of the file:
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@@
 			)
 		)
-		(property "LCSC" "C99198"
+		(property "LCSC" ""
 			(at 124.46 121.92 0)
 			(hide yes)
@@
 			)
 		)
-		(property "LCSC" "C137948"
+		(property "LCSC" ""
 			(at 119.38 68.58 90)
 			(hide yes)
@@
 			)
 		)
-		(property "LCSC" "C137948"
+		(property "LCSC" ""
 			(at 119.38 58.42 90)
 			(hide yes)
@@
 			)
 		)
-		(property "LCSC" "C137948"
+		(property "LCSC" ""
 			(at 119.38 73.66 90)
 			(hide yes)
@@
 			)
 		)
-		(property "LCSC" "C137948"
+		(property "LCSC" ""
 			(at 119.38 63.5 90)
 			(hide yes)

Commit message: update resistors to jlcpcb basic components
Parts:
- R4, R5, R6, R7: footprint Resistor_SMD:R_0402_1005Metric -> Resistor_SMD:R_0603_1608Metric; LCSC (none) -> C23228
- R8: LCSC (none) -> C25804
Changed lines of the file:
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@@
 			)
 		)
-		(property "LCSC" ""
+		(property "LCSC" "C25804"
 			(at 124.46 121.92 0)
 			(hide yes)
@@
 			)
 		)
-		(property "Footprint" "Resistor_SMD:R_0402_1005Metric"
+		(property "Footprint" "Resistor_SMD:R_0603_1608Metric"
 			(at 119.38 68.58 0)
 			(hide yes)
@@
 			)
 		)
-		(property "LCSC" ""
+		(property "LCSC" "C23228"
 			(at 119.38 68.58 90)
 			(hide yes)
@@
 			)
 		)
-		(property "Footprint" "Resistor_SMD:R_0402_1005Metric"
+		(property "Footprint" "Resistor_SMD:R_0603_1608Metric"
 			(at 119.38 58.42 0)
 			(hide yes)
@@
 			)
 		)
-		(property "LCSC" ""
+		(property "LCSC" "C23228"
 			(at 119.38 58.42 90)
 			(hide yes)
@@
 			)
 		)
-		(property "Footprint" "Resistor_SMD:R_0402_1005Metric"
+		(property "Footprint" "Resistor_SMD:R_0603_1608Metric"
 			(at 119.38 73.66 0)
 			(hide yes)
@@
 			)
 		)
-		(property "LCSC" ""
+		(property "LCSC" "C23228"
 			(at 119.38 73.66 90)
 			(hide yes)
@@
 			)
 		)
-		(property "Footprint" "Resistor_SMD:R_0402_1005Metric"
+		(property "Footprint" "Resistor_SMD:R_0603_1608Metric"
 			(at 119.38 63.5 0)
 			(hide yes)
@@
 			)
 		)
-		(property "LCSC" ""
+		(property "LCSC" "C23228"
 			(at 119.38 63.5 90)
 			(hide yes)
