File: esp32s3_breakout.kicad_sch (KiCad schematic)
At the start: 15 parts, among them J7 USB_C_Receptacle_USB2.0_16P, SW1 USAKRO UK-B0227-G4.3-B-250, SW2 USAKRO UK-B0227-G4.3-B-250, U1 ESP32-S3-WROOM-1U

Commit message: do some pcb routing
Parts:
- renumbered C30 to C29, C31 to C30, C32 to C31, C33 to C32, C34 to C33, D1 to D10, J7 to J5, R2 to R20, R15 to R21, R3 to R22, R4 to R23, U1 to U6
Changed lines of the file:
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@@
 		(in_pos_files yes)
 		(dnp no)
-		(property "Reference" "C31"
+		(property "Reference" "C30"
 			(at 68.072 50.8 0)
 			(show_name no)
@@
 			(project "gse_control_node"
 				(path "/24817451-dfe0-4b9a-9d93-7304529c9d58/df47027d-81c2-4457-b2a4-c1e06ebb5a1a"
-					(reference "C31")
+					(reference "C30")
 					(unit 1)
 				)
@@
 		(in_pos_files yes)
 		(dnp no)
-		(property "Reference" "C33"
+		(property "Reference" "C32"
 			(at 94.742 135.89 0)
 			(show_name no)
@@
 			(project "gse_control_node"
 				(path "/24817451-dfe0-4b9a-9d93-7304529c9d58/df47027d-81c2-4457-b2a4-c1e06ebb5a1a"
-					(reference "C33")
+					(reference "C32")
 					(unit 1)
 				)
@@
 		(dnp no)
 		(fields_autoplaced yes)
-		(property "Reference" "#PWR012"
+		(property "Reference" "#PWR062"
 			(at 105.41 140.97 0)
 			(hide yes)
@@
 			(project "gse_control_node"
 				(path "/24817451-dfe0-4b9a-9d93-7304529c9d58/df47027d-81c2-4457-b2a4-c1e06ebb5a1a"
-					(reference "#PWR012")
+					(reference "#PWR062")
 					(unit 1)
 				)
@@
 		(dnp no)
 		(fields_autoplaced yes)
-		(property "Reference" "#PWR015"
+		(property "Reference" "#PWR065"
 			(at 160.02 104.14 0)
 			(hide yes)
@@
 			(project "gse_control_node"
 				(path "/24817451-dfe0-4b9a-9d93-7304529c9d58/df47027d-81c2-4457-b2a4-c1e06ebb5a1a"
-					(reference "#PWR015")
+					(reference "#PWR065")
 					(unit 1)
 				)
@@
 		(dnp no)
 		(fields_autoplaced yes)
-		(property "Reference" "D1"
+		(property "Reference" "D10"
 			(at 161.29 128.5874 90)
 			(show_name no)
@@
 			(project "gse_control_node"
 				(path "/24817451-dfe0-4b9a-9d93-7304529c9d58/df47027d-81c2-4457-b2a4-c1e06ebb5a1a"
-					(reference "D1")
+					(reference "D10")
 					(unit 1)
 				)
@@
 		(in_pos_files yes)
 		(dnp no)
-		(property "Reference" "U1"
+		(property "Reference" "U6"
 			(at 111.506 49.276 0)
 			(show_name no)
@@
 			(project "gse_control_node"
 				(path "/24817451-dfe0-4b9a-9d93-7304529c9d58/df47027d-81c2-4457-b2a4-c1e06ebb5a1a"
-					(reference "U1")
+					(reference "U6")
 					(unit 1)
 				)
@@
 		(in_pos_files yes)
 		(dnp no)
-		(property "Reference" "R4"
+		(property "Reference" "R23"
 			(at 175.514 67.056 90)
 			(show_name no)
@@
 			(project "gse_control_node"
 				(path "/24817451-dfe0-4b9a-9d93-7304529c9d58/df47027d-81c2-4457-b2a4-c1e06ebb5a1a"
-					(reference "R4")
+					(reference "R23")
 					(unit 1)
 				)
@@
 		(dnp no)
 		(fields_autoplaced yes)
-		(property "Reference" "#PWR0105"
+		(property "Reference" "#PWR061"
 			(at 102.87 114.3 0)
 			(hide yes)
@@
 			(project "gse_control_node"
 				(path "/24817451-dfe0-4b9a-9d93-7304529c9d58/df47027d-81c2-4457-b2a4-c1e06ebb5a1a"
-					(reference "#PWR0105")
+					(reference "#PWR061")
 					(unit 1)
 				)
@@
 		(in_pos_files yes)
 		(dnp no)
-		(property "Reference" "C34"
+		(property "Reference" "C33"
 			(at 248.412 77.47 0)
 			(show_name no)
@@
 			(project "gse_control_node"
 				(path "/24817451-dfe0-4b9a-9d93-7304529c9d58/df47027d-81c2-4457-b2a4-c1e06ebb5a1a"
-					(reference "C34")
+					(reference "C33")
 					(unit 1)
 				)
@@
 		(in_pos_files yes)
 		(dnp no)
-		(property "Reference" "R3"
+		(property "Reference" "R22"
 			(at 175.514 59.944 90)
 			(show_name no)
@@
 			(project "gse_control_node"
 				(path "/24817451-dfe0-4b9a-9d93-7304529c9d58/df47027d-81c2-4457-b2a4-c1e06ebb5a1a"
-					(reference "R3")
+					(reference "R22")
 					(unit 1)
 				)
@@
 		(dnp no)
 		(fields_autoplaced yes)
-		(property "Reference" "J7"
+		(property "Reference" "J5"
 			(at 160.02 49.53 0)
 			(show_name no)
@@
 			(project "gse_control_node"
 				(path "/24817451-dfe0-4b9a-9d93-7304529c9d58/df47027d-81c2-4457-b2a4-c1e06ebb5a1a"
-					(reference "J7")
+					(reference "J5")
 					(unit 1)
 				)
@@
 		(in_pos_files yes)
 		(dnp no)
-		(property "Reference" "R2"
+		(property "Reference" "R20"
 			(at 78.74 53.086 0)
 			(show_name no)
@@
 			(project "gse_control_node"
 				(path "/24817451-dfe0-4b9a-9d93-7304529c9d58/df47027d-81c2-4457-b2a4-c1e06ebb5a1a"
-					(reference "R2")
+					(reference "R20")
 					(unit 1)
 				)
@@
 		(in_pos_files yes)
 		(dnp no)
-		(property "Reference" "C30"
+		(property "Reference" "C29"
 			(at 58.166 50.8 0)
 			(show_name no)
@@
 			(project "gse_control_node"
 				(path "/24817451-dfe0-4b9a-9d93-7304529c9d58/df47027d-81c2-4457-b2a4-c1e06ebb5a1a"
-					(reference "C30")
+					(reference "C29")
 					(unit 1)
 				)
@@
 		(in_pos_files yes)
 		(dnp no)
-		(property "Reference" "C32"
+		(property "Reference" "C31"
 			(at 69.088 58.674 0)
 			(show_name no)
@@
 			(project "gse_control_node"
 				(path "/24817451-dfe0-4b9a-9d93-7304529c9d58/df47027d-81c2-4457-b2a4-c1e06ebb5a1a"
-					(reference "C32")
+					(reference "C31")
 					(unit 1)
 				)
@@
 		(dnp no)
 		(fields_autoplaced yes)
-		(property "Reference" "#PWR018"
+		(property "Reference" "#PWR068"
 			(at 246.38 88.9 0)
 			(hide yes)
@@
 			(project "gse_control_node"
 				(path "/24817451-dfe0-4b9a-9d93-7304529c9d58/df47027d-81c2-4457-b2a4-c1e06ebb5a1a"
-					(reference "#PWR018")
+					(reference "#PWR068")
 					(unit 1)
 				)
@@
 		(in_pos_files yes)
 		(dnp no)
-		(property "Reference" "#PWR010"
+		(property "Reference" "#PWR059"
 			(at 74.93 69.85 0)
 			(hide yes)
@@
 			(project "gse_control_node"
 				(path "/24817451-dfe0-4b9a-9d93-7304529c9d58/df47027d-81c2-4457-b2a4-c1e06ebb5a1a"
-					(reference "#PWR010")
+					(reference "#PWR059")
 					(unit 1)
 				)
@@
 		(dnp no)
 		(fields_autoplaced yes)
-		(property "Reference" "#PWR014"
+		(property "Reference" "#PWR063"
 			(at 130.81 140.97 0)
 			(hide yes)
@@
 			(project "gse_control_node"
 				(path "/24817451-dfe0-4b9a-9d93-7304529c9d58/df47027d-81c2-4457-b2a4-c1e06ebb5a1a"
-					(reference "#PWR014")
+					(reference "#PWR063")
 					(unit 1)
 				)
@@
 		(dnp no)
 		(fields_autoplaced yes)
-		(property "Reference" "R15"
+		(property "Reference" "R21"
 			(at 160.02 121.9201 0)
 			(show_name no)
@@
 			(project "gse_control_node"
 				(path "/24817451-dfe0-4b9a-9d93-7304529c9d58/df47027d-81c2-4457-b2a4-c1e06ebb5a1a"
-					(reference "R15")
+					(reference "R21")
 					(unit 1)
 				)
@@
 		(dnp no)
 		(fields_autoplaced yes)
-		(property "Reference" "#PWR08"
+		(property "Reference" "#PWR058"
 			(at 55.88 63.5 0)
 			(hide yes)
@@
 			(project "gse_control_node"
 				(path "/24817451-dfe0-4b9a-9d93-7304529c9d58/df47027d-81c2-4457-b2a4-c1e06ebb5a1a"
-					(reference "#PWR08")
+					(reference "#PWR058")
 					(unit 1)
 				)
@@
 		(dnp no)
 		(fields_autoplaced yes)
-		(property "Reference" "#PWR0103"
+		(property "Reference" "#PWR064"
 			(at 157.48 139.7 0)
 			(hide yes)
@@
 			(project "gse_control_node"
 				(path "/24817451-dfe0-4b9a-9d93-7304529c9d58/df47027d-81c2-4457-b2a4-c1e06ebb5a1a"
-					(reference "#PWR0103")
+					(reference "#PWR064")
 					(unit 1)
 				)
@@
 		(in_pos_files yes)
 		(dnp no)
-		(property "Reference" "#PWR0104"
+		(property "Reference" "#PWR057"
 			(at 55.88 50.8 0)
 			(hide yes)
@@
 			(project "gse_control_node"
 				(path "/24817451-dfe0-4b9a-9d93-7304529c9d58/df47027d-81c2-4457-b2a4-c1e06ebb5a1a"
-					(reference "#PWR0104")
+					(reference "#PWR057")
 					(unit 1)
 				)
@@
 		(in_pos_files yes)
 		(dnp no)
-		(property "Reference" "#PWR016"
+		(property "Reference" "#PWR066"
 			(at 185.42 69.85 0)
 			(hide yes)
@@
 			(project "gse_control_node"
 				(path "/24817451-dfe0-4b9a-9d93-7304529c9d58/df47027d-81c2-4457-b2a4-c1e06ebb5a1a"
-					(reference "#PWR016")
+					(reference "#PWR066")
 					(unit 1)
 				)
@@
 		(dnp no)
 		(fields_autoplaced yes)
-		(property "Reference" "#PWR011"
+		(property "Reference" "#PWR060"
 			(at 92.71 147.32 0)
 			(hide yes)
@@
 			(project "gse_control_node"
 				(path "/24817451-dfe0-4b9a-9d93-7304529c9d58/df47027d-81c2-4457-b2a4-c1e06ebb5a1a"
-					(reference "#PWR011")
+					(reference "#PWR060")
 					(unit 1)
 				)
@@
 		(in_pos_files yes)
 		(dnp no)
-		(property "Reference" "#PWR017"
+		(property "Reference" "#PWR067"
 			(at 196.85 82.55 0)
 			(hide yes)
@@
 			(project "gse_control_node"
 				(path "/24817451-dfe0-4b9a-9d93-7304529c9d58/df47027d-81c2-4457-b2a4-c1e06ebb5a1a"
-					(reference "#PWR017")
+					(reference "#PWR067")
 					(unit 1)
 				)

Commit message: finish pcb routing
Connections:
- net 12V_POWER_GOOD: now also U6.23 (IO21)
- net ACTUATOR_1_CTL: now also U6.12 (IO8)
- net ACTUATOR_2_CTL: now also U6.10 (IO17)
- net ACTUATOR_3_CTL: now also U6.9 (IO16)
- net ACTUATOR_4_CTL: now also U6.8 (IO15)
- net DRDY1: now also U6.5 (IO5)
- net FAN_1_PWM: now also U6.33 (IO40)
- net FAN_1_TACH: now also U6.32 (IO39)
- net FAN_2_PWM: now also U6.35 (IO42)
- net FAN_2_TACH: now also U6.34 (IO41)
- net GND: now also J5.SH (SHIELD); no longer J5.S1 (SHIELD)
- net I2C_SCL: now also U6.7 (IO7)
- net I2C_SDA: now also U6.6 (IO6)
- net 5.17V_POWER_GOOD: now reaches U6.22 (IO14)
- no-connect marks 16 -> 13
Changed lines of the file:
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@@
+	)
+	(no_connect
+		(at 118.11 99.06)
+	)
+	(no_connect
+		(at 118.11 93.98)
 	)
 	(no_connect
@@
 	)
 	(no_connect
-		(at 87.63 99.06)
+		(at 118.11 101.6)
 	)
 	(no_connect
-		(at 118.11 93.98)
+		(at 87.63 68.58)
 	)
 	(no_connect
@@
 	)
 	(no_connect
-		(at 87.63 68.58)
-	)
-	(no_connect
-		(at 118.11 101.6)
-	)
-	(no_connect
 		(at 118.11 78.74)
-	)
-	(no_connect
-		(at 118.11 99.06)
 	)
 	(no_connect
@@
 		(at 175.26 87.63)
 	)
-	(no_connect
-		(at 87.63 101.6)
-	)
-	(no_connect
-		(at 118.11 60.96)
-	)
 	(wire
 		(pts
@@
 	(wire
 		(pts
+			(xy 86.36 73.66) (xy 87.63 73.66)
+		)
+		(stroke
+			(width 0)
+			(type default)
+		)
+	)
+	(wire
+		(pts
 			(xy 114.3 133.35) (xy 119.38 133.35)
 		)
@@
 	(wire
 		(pts
+			(xy 86.36 78.74) (xy 87.63 78.74)
+		)
+		(stroke
+			(width 0)
+			(type default)
+		)
+	)
+	(wire
+		(pts
 			(xy 181.61 62.23) (xy 182.88 62.23)
 		)
@@
 	(wire
 		(pts
+			(xy 118.11 86.36) (xy 119.38 86.36)
+		)
+		(stroke
+			(width 0)
+			(type default)
+		)
+	)
+	(wire
+		(pts
 			(xy 233.68 69.85) (xy 234.95 69.85)
 		)
@@
 	(wire
 		(pts
+			(xy 86.36 96.52) (xy 87.63 96.52)
+		)
+		(stroke
+			(width 0)
+			(type default)
+		)
+	)
+	(wire
+		(pts
 			(xy 233.68 74.93) (xy 246.38 74.93)
 		)
@@
 	(wire
 		(pts
+			(xy 118.11 91.44) (xy 119.38 91.44)
+		)
+		(stroke
+			(width 0)
+			(type default)
+		)
+	)
+	(wire
+		(pts
 			(xy 55.88 54.61) (xy 55.88 55.88)
 		)
@@
 	(wire
 		(pts
+			(xy 78.74 63.5) (xy 87.63 63.5)
+		)
+		(stroke
+			(width 0)
+			(type default)
+		)
+	)
+	(wire
+		(pts
 			(xy 176.53 77.47) (xy 177.8 77.47)
 		)
@@
 	(wire
 		(pts
+			(xy 86.36 99.06) (xy 87.63 99.06)
+		)
+		(stroke
+			(width 0)
+			(type default)
+		)
+	)
+	(wire
+		(pts
 			(xy 175.26 69.85) (xy 176.53 69.85)
 		)
@@
 	(wire
 		(pts
+			(xy 118.11 88.9) (xy 119.38 88.9)
+		)
+		(stroke
+			(width 0)
+			(type default)
+		)
+	)
+	(wire
+		(pts
+			(xy 86.36 101.6) (xy 87.63 101.6)
+		)
+		(stroke
+			(width 0)
+			(type default)
+		)
+	)
+	(wire
+		(pts
 			(xy 175.26 72.39) (xy 176.53 72.39)
 		)
@@
 	(wire
 		(pts
+			(xy 118.11 71.12) (xy 119.38 71.12)
+		)
+		(stroke
+			(width 0)
+			(type default)
+		)
+	)
+	(wire
+		(pts
 			(xy 246.38 81.28) (xy 246.38 82.55)
 		)
@@
 	(wire
 		(pts
+			(xy 86.36 76.2) (xy 87.63 76.2)
+		)
+		(stroke
+			(width 0)
+			(type default)
+		)
+	)
+	(wire
+		(pts
 			(xy 74.93 55.88) (xy 87.63 55.88)
 		)
@@
 	(wire
 		(pts
-			(xy 78.74 63.5) (xy 87.63 63.5)
-		)
-		(stroke
-			(width 0)
-			(type default)
-		)
-	)
-	(wire
-		(pts
 			(xy 130.81 133.35) (xy 130.81 134.62)
 		)
@@
 	(wire
 		(pts
+			(xy 118.11 83.82) (xy 119.38 83.82)
+		)
+		(stroke
+			(width 0)
+			(type default)
+		)
+	)
+	(wire
+		(pts
 			(xy 74.93 49.53) (xy 74.93 48.26)
 		)
@@
 	(wire
 		(pts
+			(xy 86.36 81.28) (xy 87.63 81.28)
+		)
+		(stroke
+			(width 0)
+			(type default)
+		)
+	)
+	(wire
+		(pts
 			(xy 92.71 133.35) (xy 93.98 133.35)
 		)
@@
 		(pts
 			(xy 118.11 66.04) (xy 119.38 66.04)
+		)
+		(stroke
+			(width 0)
+			(type default)
+		)
+	)
+	(wire
+		(pts
+			(xy 118.11 60.96) (xy 119.38 60.96)
 		)
 		(stroke
@@
 	(hierarchical_label "FAN_2_PWM"
 		(shape output)
-		(at 119.38 96.52 0)
+		(at 119.38 91.44 0)
 		(effects
 			(font
@@
 	(hierarchical_label "FAN_1_PWM"
 		(shape output)
-		(at 119.38 93.98 0)
+		(at 119.38 86.36 0)
 		(effects
 			(font
@@
 	)
 	(hierarchical_label "12V_POWER_GOOD"
-		(shape input)
-		(at 86.36 78.74 180)
-		(effects
-			(font
-				(size 1.27 1.27)
-			)
-			(justify right)
-		)
-	)
-	(hierarchical_label "DRDY1"
 		(shape input)
 		(at 119.38 71.12 0)
@@
 		)
 	)
+	(hierarchical_label "DRDY1"
+		(shape input)
+		(at 86.36 73.66 180)
+		(effects
+			(font
+				(size 1.27 1.27)
+			)
+			(justify right)
+		)
+	)
 	(hierarchical_label "ACTUATOR_2_CTL"
 		(shape output)
+		(at 119.38 60.96 0)
+		(effects
+			(font
+				(size 1.27 1.27)
+			)
+			(justify left)
+		)
+	)
+	(hierarchical_label "FAN_2_TACH"
+		(shape input)
+		(at 119.38 88.9 0)
+		(effects
+			(font
+				(size 1.27 1.27)
+			)
+			(justify left)
+		)
+	)
+	(hierarchical_label "I2C_SDA"
+		(shape bidirectional)
+		(at 86.36 76.2 180)
+		(effects
+			(font
+				(size 1.27 1.27)
+			)
+			(justify right)
+		)
+	)
+	(hierarchical_label "I2C_SCL"
+		(shape bidirectional)
+		(at 86.36 78.74 180)
+		(effects
+			(font
+				(size 1.27 1.27)
+			)
+			(justify right)
+		)
+	)
+	(hierarchical_label "5.17V_POWER_GOOD"
+		(shape input)
+		(at 86.36 96.52 180)
+		(effects
+			(font
+				(size 1.27 1.27)
+			)
+			(justify right)
+		)
+	)
+	(hierarchical_label "ACTUATOR_3_CTL"
+		(shape output)
+		(at 86.36 101.6 180)
+		(effects
+			(font
+				(size 1.27 1.27)
+			)
+			(justify right)
+		)
+	)
+	(hierarchical_label "ACTUATOR_1_CTL"
+		(shape output)
+		(at 86.36 81.28 180)
+		(effects
+			(font
+				(size 1.27 1.27)
+			)
+			(justify right)
+		)
+	)
+	(hierarchical_label "FAN_1_TACH"
+		(shape input)
 		(at 119.38 83.82 0)
 		(effects
@@
 		)
 	)
-	(hierarchical_label "FAN_2_TACH"
-		(shape input)
-		(at 119.38 101.6 0)
+	(hierarchical_label "ACTUATOR_4_CTL"
+		(shape output)
+		(at 86.36 99.06 180)
 		(effects
 			(font
 				(size 1.27 1.27)
 			)
-			(justify left)
-		)
-	)
-	(hierarchical_label "I2C_SDA"
-		(shape bidirectional)
-		(at 86.36 83.82 180)
-		(effects
-			(font
-				(size 1.27 1.27)
-			)
 			(justify right)
-		)
-	)
-	(hierarchical_label "I2C_SCL"
-		(shape bidirectional)
-		(at 86.36 86.36 180)
-		(effects
-			(font
-				(size 1.27 1.27)
-			)
-			(justify right)
-		)
-	)
-	(hierarchical_label "5.3V_POWER_GOOD"
-		(shape input)
-		(at 86.36 81.28 180)
-		(effects
-			(font
-				(size 1.27 1.27)
-			)
-			(justify right)
-		)
-	)
-	(hierarchical_label "ACTUATOR_3_CTL"
-		(shape output)
-		(at 119.38 86.36 0)
-		(effects
-			(font
-				(size 1.27 1.27)
-			)
-			(justify left)
-		)
-	)
-	(hierarchical_label "ACTUATOR_1_CTL"
-		(shape output)
-		(at 119.38 81.28 0)
-		(effects
-			(font
-				(size 1.27 1.27)
-			)
-			(justify left)
-		)
-	)
-	(hierarchical_label "FAN_1_TACH"
-		(shape input)
-		(at 119.38 99.06 0)
-		(effects
-			(font
-				(size 1.27 1.27)
-			)
-			(justify left)
-		)
-	)
-	(hierarchical_label "ACTUATOR_4_CTL"
-		(shape output)
-		(at 119.38 88.9 0)
-		(effects
-			(font
-				(size 1.27 1.27)
-			)
-			(justify left)
 		)
 	)
@@
 			)
 		)
-		(pin "S1"
+		(pin "SH"
 		)
 		(pin "B1"

Commit message: remove unneccesary component fields
Parts:
- C29: Dielectric X5R or X7R -> (none); LCSC C602037 -> (none)
- C30, C32, C33: value 0.1μF -> 100nF; LCSC C307331 -> (none); MPN CL05B104KO5NNNC -> (none)
- C31: Dielectric X5R or X7R -> (none); LCSC C29936 -> (none)
- R20: value 10k -> 10kΩ; footprint Resistor_SMD:R_0402_1005Metric -> Resistor_SMD:R_0603_1608Metric
- R21: value 1k -> 1kΩ
- R22, R23: value 5.1k -> 5.1kΩ
Connections:
- no-connect marks 13 -> 21

Commit message: add all lcsc part numbers
Parts:
- C29: LCSC (none) -> C45783
- C30, C32, C33: LCSC (none) -> C85858
- C31: LCSC (none) -> C29936
- R20: LCSC (none) -> C99198
- R21: LCSC (none) -> C106235
- R22, R23: LCSC (none) -> C105872
Changed lines of the file:
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@@
 			)
 		)
-		(property "LCSC" ""
+		(property "LCSC" "C85858"
 			(at 66.04 52.07 0)
 			(hide yes)
@@
 			)
 		)
-		(property "LCSC" ""
+		(property "LCSC" "C85858"
 			(at 92.71 137.16 0)
 			(hide yes)
@@
 			)
 		)
+		(property "LCSC" "C105872"
+			(at 179.07 64.77 90)
+			(hide yes)
+			(show_name no)
+			(do_not_autoplace no)
+			(effects
+				(font
+					(size 1.27 1.27)
+				)
+			)
+		)
 		(pin "2"
 		)
@@
 			)
 		)
-		(property "LCSC" ""
+		(property "LCSC" "C85858"
 			(at 246.38 78.74 0)
 			(hide yes)
@@
 		(property "Description" "Resistor, small US symbol"
 			(at 179.07 62.23 0)
+			(hide yes)
+			(show_name no)
+			(do_not_autoplace no)
+			(effects
+				(font
+					(size 1.27 1.27)
+				)
+			)
+		)
+		(property "LCSC" "C105872"
+			(at 179.07 62.23 90)
 			(hide yes)
 			(show_name no)
@@
 			)
 		)
+		(property "LCSC" "C99198"
+			(at 74.93 52.07 0)
+			(hide yes)
+			(show_name no)
+			(do_not_autoplace no)
+			(effects
+				(font
+					(size 1.27 1.27)
+				)
+			)
+		)
 		(pin "2"
 		)
@@
 			)
 		)
-		(property "LCSC" ""
+		(property "LCSC" "C45783"
 			(at 55.88 52.07 0)
 			(hide yes)
@@
 			)
 		)
-		(property "LCSC" ""
+		(property "LCSC" "C29936"
 			(at 74.93 59.69 0)
 			(hide yes)
@@
 			(at 157.48 120.65 0)
 			(hide yes)
+			(show_name no)
+			(do_not_autoplace no)
+			(effects
+				(font
+					(size 1.27 1.27)
+				)
+			)
+		)
+		(property "LCSC" "C106235"
+			(at 157.48 120.65 0)
+			(hide yes)

Commit message: switch to esp32-s3-wroom-1
Parts:
- U6: value ESP32-S3-WROOM-1U -> ESP32-S3-WROOM-1; footprint RF_Module:ESP32-S3-WROOM-1U -> RF_Module:ESP32-S3-WROOM-1; LCSC C3013946 -> C2913202
Changed lines of the file:
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@@
 			)
 		)
-		(property "Value" "ESP32-S3-WROOM-1U"
+		(property "Value" "ESP32-S3-WROOM-1"
 			(at 104.14 51.816 0)
 			(show_name no)
@@
 			)
 		)
-		(property "Footprint" "RF_Module:ESP32-S3-WROOM-1U"
+		(property "Footprint" "RF_Module:ESP32-S3-WROOM-1"
 			(at 102.87 76.2 0)
 			(hide yes)
@@
 			)
 		)
-		(property "LCSC" "C3013946"
+		(property "LCSC" "C2913202"
 			(at 102.87 78.74 0)
 			(hide yes)

Commit message: update all capacitors to jlcpcb basic components
Parts:
- C30, C32, C33: LCSC C85858 -> C307331
- C31: LCSC C29936 -> C15849
Changed lines of the file:
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@@
 			)
 		)
-		(property "LCSC" "C85858"
+		(property "LCSC" "C307331"
 			(at 66.04 52.07 0)
 			(hide yes)
@@
 			)
 		)
-		(property "LCSC" "C85858"
+		(property "LCSC" "C307331"
 			(at 92.71 137.16 0)
 			(hide yes)
@@
 			)
 		)
-		(property "LCSC" "C85858"
+		(property "LCSC" "C307331"
 			(at 246.38 78.74 0)
 			(hide yes)
@@
 			)
 		)
-		(property "LCSC" "C29936"
+		(property "LCSC" "C15849"
 			(at 74.93 59.69 0)
 			(hide yes)

Commit message: add a 12v testpoint
Parts:
- R20: LCSC C99198 -> (none)
- R21: LCSC C106235 -> (none)
- R22, R23: LCSC C105872 -> (none)
Changed lines of the file:
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@@
 			)
 		)
-		(property "LCSC" "C105872"
+		(property "LCSC" ""
 			(at 179.07 64.77 90)
 			(hide yes)
@@
 			)
 		)
-		(property "LCSC" "C105872"
+		(property "LCSC" ""
 			(at 179.07 62.23 90)
 			(hide yes)
@@
 			)
 		)
-		(property "LCSC" "C99198"
+		(property "LCSC" ""
 			(at 74.93 52.07 0)
 			(hide yes)
@@
 			)
 		)
-		(property "LCSC" "C106235"
+		(property "LCSC" ""
 			(at 157.48 120.65 0)
 			(hide yes)

Commit message: update resistors to jlcpcb basic components
Parts:
- R20: LCSC (none) -> C25804
- R21: footprint Resistor_SMD:R_0402_1005Metric -> Resistor_SMD:R_0603_1608Metric; LCSC (none) -> C21190
- R22, R23: footprint Resistor_SMD:R_0402_1005Metric -> Resistor_SMD:R_0603_1608Metric
Changed lines of the file:
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@@
 			)
 		)
-		(property "Footprint" "Resistor_SMD:R_0402_1005Metric"
+		(property "Footprint" "Resistor_SMD:R_0603_1608Metric"
 			(at 179.07 64.77 0)
 			(hide yes)
@@
 			)
 		)
-		(property "Footprint" "Resistor_SMD:R_0402_1005Metric"
+		(property "Footprint" "Resistor_SMD:R_0603_1608Metric"
 			(at 179.07 62.23 0)
 			(hide yes)
@@
 			)
 		)
-		(property "LCSC" ""
+		(property "LCSC" "C25804"
 			(at 74.93 52.07 0)
 			(hide yes)
@@
 			)
 		)
-		(property "Footprint" "Resistor_SMD:R_0402_1005Metric"
+		(property "Footprint" "Resistor_SMD:R_0603_1608Metric"
 			(at 157.48 120.65 0)
 			(hide yes)
@@
 			)
 		)
-		(property "LCSC" ""
+		(property "LCSC" "C21190"
 			(at 157.48 120.65 0)
 			(hide yes)
