File: gse_control_node/actuator_control.kicad_sch (KiCad schematic)
At the start: 5 parts, among them J7 Conn_01x02, Q2 BSS138

Commit message: finish control board routing
Parts:
- added D15, D19, D23: SK44BL, Diode_SMD:D_SMB, symbol Device:D_Schottky_Small
- added J15, J22, J26: Conn_01x02, Connector_Molex:Molex_Micro-Fit_3.0_43650-0215_1x02_P3.00mm_Vertical, symbol Connector_Generic:Conn_01x02
- added Q13, Q17, Q7: BSS138, Package_TO_SOT_SMD:SOT-23-3, symbol dk_Transistors-FETs-MOSFETs-Single:BSS138
- added R33, R57, R65: 100kΩ, Resistor_SMD:R_0603_1608Metric, symbol Device:R_Small_US
- added R36, R58, R66: 100Ω, Resistor_SMD:R_0603_1608Metric, symbol Device:R_Small_US
Connections:
- net +24V: now also D15.1 (K), D19.1 (K), D23.1 (K), J15.1 (Pin_1), J22.1 (Pin_1), J26.1 (Pin_1)
- net GND: now also Q13.2 (S), Q17.2 (S), Q7.2 (S), R33.2, R57.2, R65.2
- net ACTUATOR_CTL renamed ACT1_CTL
- new net: D15.2 (A), J15.2 (Pin_2), Q7.3 (D)
- new net: Q13.1 (G), R58.2
- new net: D19.2 (A), J22.2 (Pin_2), Q13.3 (D)
- new net: Q17.1 (G), R66.2
- new net: D23.2 (A), J26.2 (Pin_2), Q17.3 (D)
- new net: Q7.1 (G), R36.2
- new net ACT2_CTL: R33.1, R36.1
- new net ACT3_CTL: R57.1, R58.1
- new net ACT4_CTL: R65.1, R66.1
Other:
- moved on the sheet: D11, J7, Q2, R24, R25

Commit message: updates for manufacturing
Parts:
- D11, D15, D19, D23, J15, J22, J26, J7, Q13, Q17, Q2, Q7: now in the parts list
- R24, R36, R58, R66: value 100Ω -> 100
- R25, R33, R57, R65: value 100kΩ -> 100k
Changed lines of the file:
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@@
 		(body_style 1)
 		(exclude_from_sim no)
-		(in_bom no)
-		(on_board yes)
-		(in_pos_files no)
+		(in_bom yes)
+		(on_board yes)
+		(in_pos_files yes)
 		(dnp no)
 		(fields_autoplaced yes)
@@
 		(body_style 1)
 		(exclude_from_sim no)
-		(in_bom no)
-		(on_board yes)
-		(in_pos_files no)
+		(in_bom yes)
+		(on_board yes)
+		(in_pos_files yes)
 		(dnp no)
 		(fields_autoplaced yes)
@@
 		(body_style 1)
 		(exclude_from_sim no)
-		(in_bom no)
-		(on_board yes)
-		(in_pos_files no)
+		(in_bom yes)
+		(on_board yes)
+		(in_pos_files yes)
 		(dnp no)
 		(property "Reference" "D11"
@@
 		(body_style 1)
 		(exclude_from_sim no)
-		(in_bom no)
-		(on_board yes)
-		(in_pos_files no)
+		(in_bom yes)
+		(on_board yes)
+		(in_pos_files yes)
 		(dnp no)
 		(fields_autoplaced yes)
@@
 			)
 		)
-		(property "Value" "100kΩ"
+		(property "Value" "100k"
 			(at 48.768 52.578 0)
 			(show_name no)
@@
 			)
 		)
-		(property "Value" "100kΩ"
+		(property "Value" "100k"
 			(at 127.508 52.578 0)
 			(show_name no)
@@
 			)
 		)
-		(property "Value" "100kΩ"
+		(property "Value" "100k"
 			(at 127.508 90.678 0)
 			(show_name no)
@@
 		(body_style 1)
 		(exclude_from_sim no)
-		(in_bom no)
-		(on_board yes)
-		(in_pos_files no)
+		(in_bom yes)
+		(on_board yes)
+		(in_pos_files yes)
 		(dnp no)
 		(property "Reference" "D19"
@@
 		(body_style 1)
 		(exclude_from_sim no)
-		(in_bom no)
-		(on_board yes)
-		(in_pos_files no)
+		(in_bom yes)
+		(on_board yes)
+		(in_pos_files yes)
 		(dnp no)
 		(fields_autoplaced yes)
@@
 			)
 		)
-		(property "Value" "100kΩ"
+		(property "Value" "100k"
 			(at 48.768 90.678 0)
 			(show_name no)
@@
 		(body_style 1)
 		(exclude_from_sim no)
-		(in_bom no)
-		(on_board yes)
-		(in_pos_files no)
+		(in_bom yes)
+		(on_board yes)
+		(in_pos_files yes)
 		(dnp no)
 		(fields_autoplaced yes)
@@
 			)
 		)
-		(property "Value" "100Ω"
+		(property "Value" "100"
 			(at 129.286 82.804 90)
 			(show_name no)
@@
 		(body_style 1)
 		(exclude_from_sim no)
-		(in_bom no)
-		(on_board yes)
-		(in_pos_files no)
+		(in_bom yes)
+		(on_board yes)
+		(in_pos_files yes)
 		(dnp no)
 		(fields_autoplaced yes)
@@
 			)
 		)
-		(property "Value" "100Ω"
+		(property "Value" "100"
 			(at 50.546 44.704 90)
 			(show_name no)
@@
 		(body_style 1)
 		(exclude_from_sim no)
-		(in_bom no)
-		(on_board yes)
-		(in_pos_files no)
+		(in_bom yes)
+		(on_board yes)
+		(in_pos_files yes)
 		(dnp no)
 		(property "Reference" "D15"
@@
 		(body_style 1)
 		(exclude_from_sim no)
-		(in_bom no)
-		(on_board yes)
-		(in_pos_files no)
+		(in_bom yes)
+		(on_board yes)
+		(in_pos_files yes)
 		(dnp no)
 		(property "Reference" "D23"
@@
 		(body_style 1)
 		(exclude_from_sim no)
-		(in_bom no)
-		(on_board yes)
-		(in_pos_files no)
+		(in_bom yes)
+		(on_board yes)
+		(in_pos_files yes)
 		(dnp no)
 		(fields_autoplaced yes)
@@
 		(body_style 1)
 		(exclude_from_sim no)
-		(in_bom no)
-		(on_board yes)
-		(in_pos_files no)
+		(in_bom yes)
+		(on_board yes)
+		(in_pos_files yes)
 		(dnp no)
 		(fields_autoplaced yes)
@@
 			)
 		)
-		(property "Value" "100Ω"
+		(property "Value" "100"
 			(at 50.546 82.804 90)
 			(show_name no)
@@
 			)
 		)
-		(property "Value" "100Ω"
+		(property "Value" "100"
 			(at 129.286 44.704 90)
 			(show_name no)
