File: gse_control_node/adc_filtering.kicad_sch (KiCad schematic)
At the start: 16 parts, among them U1 ADS112C04

Commit message: updates for manufacturing
Parts:
- R8: value 10kΩ -> 10k
Changed lines of the file:
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@@
 			)
 		)
-		(property "Value" "10kΩ"
+		(property "Value" "10k"
 			(at 124.46 119.126 90)
 			(show_name no)
