File: gse_control_node/adc_filtering.kicad_sch (KiCad schematic)
At the start: 16 parts, among them U1 ADS112C04

Commit message: Heater/ignitor control (#2)
* update project to kicad v10

* remove thermistors from board

* rename project to be more descriptive

* fix load cell connector

* switch to on-board esp32s3

* fix fan header footprint

* update buck converter components and add reverse polarity protection

* do some pcb routing

* finish pcb routing

* remove unneccesary component fields

* add all lcsc part numbers

* add readme

* add thermal reliefs on bottom power planes

* give more clearance for load cell connector from edge of board

* fix 5.17V buck switch node net name

* switch to esp32-s3-wroom-1

* update some routing and put ground pour on top layer to avoid warping

* update silkscreen

* update all capacitors to jlcpcb basic components

* add a 12v testpoint

* update resistors to jlcpcb basic components

* fix copper pour priorities

* move up ads112c04 capacitors further from pins for easier handsoldering

* remove some extended components from bom (to be handsoldered)

* update screw terminal footprint

* add tachometer pullup and pwm low side fet for fans

* organize hierarchical sheet page numbers

* add heater connectors

* add heater power regulation for fet switching

* seperate board directories and finish heater driver routing

* add relay to heater board for estop and do some ignitor board routing

* finish ignitor board routing

* finish control board routing

* updates for manufacturing

* remove leftover files

* improve silkscreening on ignitor board and add connector for keyswitch

* make gitignore ignore production dir recursively
Parts:
- R8: value 10kΩ -> 10k
