File: gse_control_node/esp32s3_breakout.kicad_sch (KiCad schematic)
At the start: 15 parts, among them J5 USB_C_Receptacle_USB2.0_16P, SW1 USAKRO UK-B0227-G4.3-B-250, SW2 USAKRO UK-B0227-G4.3-B-250, U6 ESP32-S3-WROOM-1

Commit message: finish control board routing
Parts:
- U6: value ESP32-S3-WROOM-1 -> ESP32-S3-WROOM-1U; footprint RF_Module:ESP32-S3-WROOM-1 -> RF_Module:ESP32-S3-WROOM-1U
Connections:
- net I2C_SCL: now also U6.6 (IO6); no longer U6.7 (IO7)
- net I2C_SDA: now also U6.7 (IO7); no longer U6.6 (IO6)
- net WIFI_IND: now also U6.31 (IO38); no longer U6.39 (IO1)
- net DRDY3: now reaches U6.17 (IO9)
- net DRDY4: now reaches U6.18 (IO10)
- net IGN_PRIME_CTL: now reaches U6.19 (IO11)
- net IGN_RUN_CTL: now reaches U6.20 (IO12)
- net SAFE24_CTL: now reaches U6.21 (IO13)
- net HEAT2_PWM: now reaches U6.24 (IO47)
- net HEAT2_ESTOP: now reaches U6.25 (IO48)
- net FAN3_TACH: now reaches U6.38 (IO2)
- net DRDY2: now reaches U6.4 (IO4)
- net 12V_POWER_GOOD renamed HEAT1_ESTOP
- net 5.17V_POWER_GOOD renamed HEAT1_PWM
- net FAN_1_PWM renamed FAN1_PWM
- net FAN_1_TACH renamed FAN1_TACH
- net FAN_2_PWM renamed FAN2_PWM
- net FAN_2_TACH renamed FAN2_TACH
- new net FAN3_PWM: U6.39 (IO1)
- no-connect marks 21 -> 11
Other:
- moved on the sheet: C29, C30, C31, R20

Commit message: updates for manufacturing
Parts:
- CR1, SW1, SW2, U6: now in the parts list
- R20: value 10kΩ -> 10k
- R21: value 1kΩ -> 1k
- R22, R23: value 5.1kΩ -> 5.1k
Changed lines of the file:
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@@
 		(body_style 1)
 		(exclude_from_sim no)
-		(in_bom no)
-		(on_board yes)
-		(in_pos_files no)
+		(in_bom yes)
+		(on_board yes)
+		(in_pos_files yes)
 		(dnp no)
 		(property "Reference" "U6"
@@
 		(body_style 1)
 		(exclude_from_sim no)
-		(in_bom no)
-		(on_board yes)
-		(in_pos_files no)
+		(in_bom yes)
+		(on_board yes)
+		(in_pos_files yes)
 		(dnp no)
 		(fields_autoplaced yes)
@@
 			)
 		)
-		(property "Value" "5.1kΩ"
+		(property "Value" "5.1k"
 			(at 179.832 67.056 90)
 			(show_name no)
@@
 		(body_style 1)
 		(exclude_from_sim no)
-		(in_bom no)
-		(on_board yes)
-		(in_pos_files no)
+		(in_bom yes)
+		(on_board yes)
+		(in_pos_files yes)
 		(dnp no)
 		(property "Reference" "SW1"
@@
 			)
 		)
-		(property "Value" "5.1kΩ"
+		(property "Value" "5.1k"
 			(at 179.832 59.944 90)
 			(show_name no)
@@
 			)
 		)
-		(property "Value" "10kΩ"
+		(property "Value" "10k"
 			(at 74.676 51.054 0)
 			(show_name no)
@@
 			)
 		)
-		(property "Value" "1kΩ"
+		(property "Value" "1k"
 			(at 160.02 119.3801 0)
 			(show_name no)
@@
 		(body_style 1)
 		(exclude_from_sim no)
-		(in_bom no)
-		(on_board yes)
-		(in_pos_files no)
+		(in_bom yes)
+		(on_board yes)
+		(in_pos_files yes)
 		(dnp no)
 		(property "Reference" "SW2"
