File: gse_control_node/esp32s3_breakout.kicad_sch (KiCad schematic)
At the start: 15 parts, among them J5 USB_C_Receptacle_USB2.0_16P, SW1 USAKRO UK-B0227-G4.3-B-250, SW2 USAKRO UK-B0227-G4.3-B-250, U6 ESP32-S3-WROOM-1

Commit message: Heater/ignitor control (#2)
* update project to kicad v10

* remove thermistors from board

* rename project to be more descriptive

* fix load cell connector

* switch to on-board esp32s3

* fix fan header footprint

* update buck converter components and add reverse polarity protection

* do some pcb routing

* finish pcb routing

* remove unneccesary component fields

* add all lcsc part numbers

* add readme

* add thermal reliefs on bottom power planes

* give more clearance for load cell connector from edge of board

* fix 5.17V buck switch node net name

* switch to esp32-s3-wroom-1

* update some routing and put ground pour on top layer to avoid warping

* update silkscreen

* update all capacitors to jlcpcb basic components

* add a 12v testpoint

* update resistors to jlcpcb basic components

* fix copper pour priorities

* move up ads112c04 capacitors further from pins for easier handsoldering

* remove some extended components from bom (to be handsoldered)

* update screw terminal footprint

* add tachometer pullup and pwm low side fet for fans

* organize hierarchical sheet page numbers

* add heater connectors

* add heater power regulation for fet switching

* seperate board directories and finish heater driver routing

* add relay to heater board for estop and do some ignitor board routing

* finish ignitor board routing

* finish control board routing

* updates for manufacturing

* remove leftover files

* improve silkscreening on ignitor board and add connector for keyswitch

* make gitignore ignore production dir recursively
Parts:
- CR1, SW1, SW2: now in the parts list
- R20: value 10kΩ -> 10k
- R21: value 1kΩ -> 1k
- R22, R23: value 5.1kΩ -> 5.1k
- U6: value ESP32-S3-WROOM-1 -> ESP32-S3-WROOM-1U; footprint RF_Module:ESP32-S3-WROOM-1 -> RF_Module:ESP32-S3-WROOM-1U; now in the parts list
Connections:
- net I2C_SCL: now also U6.6 (IO6); no longer U6.7 (IO7)
- net I2C_SDA: now also U6.7 (IO7); no longer U6.6 (IO6)
- net WIFI_IND: now also U6.31 (IO38); no longer U6.39 (IO1)
- net DRDY3: now reaches U6.17 (IO9)
- net DRDY4: now reaches U6.18 (IO10)
- net IGN_PRIME_CTL: now reaches U6.19 (IO11)
- net IGN_RUN_CTL: now reaches U6.20 (IO12)
- net SAFE24_CTL: now reaches U6.21 (IO13)
- net HEAT2_PWM: now reaches U6.24 (IO47)
- net HEAT2_ESTOP: now reaches U6.25 (IO48)
- net FAN3_TACH: now reaches U6.38 (IO2)
- net DRDY2: now reaches U6.4 (IO4)
- net 12V_POWER_GOOD renamed HEAT1_ESTOP
- net 5.17V_POWER_GOOD renamed HEAT1_PWM
- net FAN_1_PWM renamed FAN1_PWM
- net FAN_1_TACH renamed FAN1_TACH
- net FAN_2_PWM renamed FAN2_PWM
- net FAN_2_TACH renamed FAN2_TACH
- new net FAN3_PWM: U6.39 (IO1)
- no-connect marks 21 -> 11
Other:
- moved on the sheet: C29, C30, C31, R20
