File: gse_control_node/gse_control_node.kicad_pcb (KiCad board)
At the start: 4 copper layers, 65 x 65 mm, 127 parts, among them J1 Screw_Terminal_01x02, J10 Conn_01x02, J2 Conn_01x04, J3 Conn_01x04, J4 Conn_02x01, J5 USB_C_Receptacle_USB2.0_16P, J6 Conn_01x04, J7 Conn_01x02, J8 Conn_01x02, J9 Conn_01x02, Q1 DMP6023LE-13, Q2 BSS138, Q3 BSS138, Q4 BSS138, Q5 BSS138, Q6 BSS138, Q7 BSS138, SW1 USAKRO UK-B0227-G4.3-B-250, SW2 USAKRO UK-B0227-G4.3-B-250, U1 ADS112C04, U2 LMR33630BDDA, U3 LMR33630BDDA, U4 TPS78533QKVURQ1, U5 TPS78450QDBVRQ1, U6 ESP32-S3-WROOM-1, U7 LM66200

Commit message: finish control board routing
Parts:
- removed C15: 100uF, Capacitor_SMD:CP_Elec_10x10
- removed J1: Screw_Terminal_01x02, TerminalBlock_CUI:TerminalBlock_CUI_TB007-508-02_1x02_P5.08mm_Horizontal
- removed J10, J8, J9: Conn_01x02, Connector_Molex:Molex_Micro-Fit_3.0_43650-0215_1x02_P3.00mm_Vertical
- removed J6: Conn_01x04, Connector_Molex:Molex_KK-254_AE-6410-04A_1x04_P2.54mm_Vertical
- removed Q3, Q4, Q5: BSS138, Package_TO_SOT_SMD:SOT-23-3
- removed R10, R11: 100kΩ, Resistor_SMD:R_0603_1608Metric
- added C37: 100nF, Capacitor_SMD:C_0402_1005Metric, F.Cu at (150.8, 108.9)
- added C38: 100nF, Capacitor_SMD:C_0402_1005Metric, F.Cu at (150.8, 107.0)
- added C39: 220nF, Capacitor_SMD:C_0402_1005Metric, F.Cu at (164.8, 113.1)
- added C40: 220nF, Capacitor_SMD:C_0402_1005Metric, F.Cu at (164.8, 109.1)
- added C41: 220nF, Capacitor_SMD:C_0402_1005Metric, F.Cu at (164.8, 111.1)
- added C42: 220nF, Capacitor_SMD:C_0402_1005Metric, F.Cu at (164.8, 107.1)
- added C43: 100nF, Capacitor_SMD:C_0402_1005Metric, F.Cu at (159.1, 117.2)
- added C44: 100nF, Capacitor_SMD:C_0402_1005Metric, F.Cu at (159.1, 119.2)
- added C45: 220nF, Capacitor_SMD:C_0402_1005Metric, F.Cu at (144.6, 117.9)
- added C46: 220nF, Capacitor_SMD:C_0402_1005Metric, F.Cu at (165.7, 117.9)
- added C47: 220nF, Capacitor_SMD:C_0402_1005Metric, F.Cu at (144.6, 119.1)
- added C48: 220nF, Capacitor_SMD:C_0402_1005Metric, F.Cu at (165.7, 119.1)
- added C49: 100nF, Capacitor_SMD:C_0402_1005Metric, F.Cu at (133.4, 117.2)
- added C50: 100nF, Capacitor_SMD:C_0402_1005Metric, F.Cu at (133.4, 119.2)
- added C51: 220nF, Capacitor_SMD:C_0402_1005Metric, F.Cu at (118.1, 118.0)
- added C52: 220nF, Capacitor_SMD:C_0402_1005Metric, F.Cu at (140.0, 117.9)
- added C53: 220nF, Capacitor_SMD:C_0402_1005Metric, F.Cu at (118.1, 119.2)
- added C54: 220nF, Capacitor_SMD:C_0402_1005Metric, F.Cu at (140.0, 119.1)
- added C55: 100uF, Capacitor_THT:CP_Radial_D8.0mm_P5.00mm, F.Cu at (146.4, 54.1)
- added D15: SK44BL, Diode_SMD:D_SMB, F.Cu at (163.0, 68.1)
- added D16: BAT54SW, Package_TO_SOT_SMD:SOT-323_SC-70, F.Cu at (161.7, 106.2)
- added D17: BAT54SW, Package_TO_SOT_SMD:SOT-323_SC-70, F.Cu at (148.2, 117.1)
- added D18: BAT54SW, Package_TO_SOT_SMD:SOT-323_SC-70, F.Cu at (162.0, 117.1)
- added D19: SK44BL, Diode_SMD:D_SMB, F.Cu at (163.0, 76.6)
- added D20: BAT54SW, Package_TO_SOT_SMD:SOT-323_SC-70, F.Cu at (148.2, 119.9)
- added D21: BAT54SW, Package_TO_SOT_SMD:SOT-323_SC-70, F.Cu at (162.0, 119.9)
- added D22: BAT54SW, Package_TO_SOT_SMD:SOT-323_SC-70, F.Cu at (122.2, 117.2)
- added D23: SK44BL, Diode_SMD:D_SMB, F.Cu at (163.0, 85.1)
- added D24: BAT54SW, Package_TO_SOT_SMD:SOT-323_SC-70, F.Cu at (136.3, 117.1)
- added D25: BAT54SW, Package_TO_SOT_SMD:SOT-323_SC-70, F.Cu at (122.2, 120.0)
- added D26: BAT54SW, Package_TO_SOT_SMD:SOT-323_SC-70, F.Cu at (136.3, 119.9)
- added J11: Conn_01x04, Connector_Molex:Molex_KK-254_AE-6410-04A_1x04_P2.54mm_Vertical, F.Cu at (115.9, 94.1)
- added J12: Conn_02x04_Counter_Clockwise, Connector_Molex:Molex_Micro-Fit_3.0_43045-0812_2x04_P3.00mm_Vertical, F.Cu at (152.1, 128.4)
- added J13: Conn_02x05_Counter_Clockwise, Connector_Molex:Molex_Micro-Fit_3.0_43045-1012_2x05_P3.00mm_Vertical, F.Cu at (165.9, 126.6)
- added J14: Conn_02x04_Counter_Clockwise, Connector_Molex:Molex_Micro-Fit_3.0_43045-0812_2x04_P3.00mm_Vertical, F.Cu at (130.2, 128.4)
- added J15: Conn_01x02, Connector_Molex:Molex_Micro-Fit_3.0_43650-0215_1x02_P3.00mm_Vertical, F.Cu at (169.2, 67.7)
- added J16: CTL_Conn, Connector_Molex:Molex_Micro-Fit_3.0_43045-0612_2x03_P3.00mm_Vertical, F.Cu at (152.1, 139.6)
- added J17: CTL_Conn, Connector_Molex:Molex_Micro-Fit_3.0_43045-0612_2x03_P3.00mm_Vertical, F.Cu at (130.2, 139.6)
- added J18: Conn_01x04, Connector_Molex:Molex_KK-254_AE-6410-04A_1x04_P2.54mm_Vertical, F.Cu at (115.9, 106.1)
- added J22: Conn_01x02, Connector_Molex:Molex_Micro-Fit_3.0_43650-0215_1x02_P3.00mm_Vertical, F.Cu at (169.2, 76.2)
- added J26: Conn_01x02, Connector_Molex:Molex_Micro-Fit_3.0_43650-0215_1x02_P3.00mm_Vertical, F.Cu at (169.2, 84.7)
- added Q10: BSS138, Package_TO_SOT_SMD:SOT-23-3, F.Cu at (121.6, 109.3)
- added Q13: BSS138, Package_TO_SOT_SMD:SOT-23-3, F.Cu at (158.8, 75.1)
- added Q17: BSS138, Package_TO_SOT_SMD:SOT-23-3, F.Cu at (158.8, 83.6)
- added Q8: BSS138, Package_TO_SOT_SMD:SOT-23-3, F.Cu at (121.1, 99.4)
- added R38: 10k, Resistor_SMD:R_0603_1608Metric, F.Cu at (157.7, 127.5)
- added R39: 10k, Resistor_SMD:R_0603_1608Metric, F.Cu at (139.6, 114.9)
- added R40: 10k, Resistor_SMD:R_0603_1608Metric, F.Cu at (157.7, 123.7)
- added R41: 10k, Resistor_SMD:R_0603_1608Metric, F.Cu at (135.4, 123.0)
- added R42: 10k, Resistor_SMD:R_0603_1608Metric, F.Cu at (135.4, 128.4)
- added R43: 10k, Resistor_SMD:R_0603_1608Metric, F.Cu at (115.2, 120.6)
- added R44: 10k, Resistor_SMD:R_0603_1608Metric, F.Cu at (145.0, 114.9)
- added R45: 10k, Resistor_SMD:R_0603_1608Metric, F.Cu at (115.2, 116.6)
- added R46: 10kΩ, Resistor_SMD:R_0603_1608Metric, F.Cu at (121.0, 96.5)
- added R47: 100Ω, Resistor_SMD:R_0603_1608Metric, F.Cu at (120.4, 103.3)
- added R48: 100kΩ, Resistor_SMD:R_0603_1608Metric, F.Cu at (122.0, 103.3)
- added R49: 680, Resistor_SMD:R_0603_1608Metric, F.Cu at (145.0, 116.5)
- added R50: 680, Resistor_SMD:R_0603_1608Metric, F.Cu at (145.0, 120.5)
- added R51: 680, Resistor_SMD:R_0603_1608Metric, F.Cu at (165.2, 120.5)
- added R52: 10kΩ, Resistor_SMD:R_0603_1608Metric, F.Cu at (122.1, 106.2)
- added R53: 100Ω, Resistor_SMD:R_0603_1608Metric, F.Cu at (120.9, 113.1)
- added R54: 100kΩ, Resistor_SMD:R_0603_1608Metric, F.Cu at (122.5, 113.1)
- added R55: 680, Resistor_SMD:R_0603_1608Metric, F.Cu at (165.2, 116.5)
- added R56: 10kΩ, Resistor_SMD:R_0603_1608Metric, F.Cu at (151.8, 114.2)
- added R57: 100kΩ, Resistor_SMD:R_0603_1608Metric, F.Cu at (159.1, 79.6)
- added R58: 100Ω, Resistor_SMD:R_0603_1608Metric, F.Cu at (159.1, 78.0)
- added R59: 3.3kΩ, Resistor_SMD:R_0603_1608Metric, F.Cu at (130.6, 114.2)
- added R60: 680, Resistor_SMD:R_0603_1608Metric, F.Cu at (118.5, 116.6)
- added R61: 680, Resistor_SMD:R_0603_1608Metric, F.Cu at (118.5, 120.6)
- added R62: 680, Resistor_SMD:R_0603_1608Metric, F.Cu at (139.6, 120.5)
- added R63: 680, Resistor_SMD:R_0603_1608Metric, F.Cu at (139.6, 116.5)
- added R64: 10kΩ, Resistor_SMD:R_0603_1608Metric, F.Cu at (125.8, 114.2)
- added R65: 100kΩ, Resistor_SMD:R_0603_1608Metric, F.Cu at (159.1, 88.1)
- added R66: 100Ω, Resistor_SMD:R_0603_1608Metric, F.Cu at (159.1, 86.5)
- added U10: ADS112C04, Package_SO:TSSOP-16_4.4x5mm_P0.65mm, F.Cu at (128.2, 118.2)
- added U8: ADS112C04, Package_SO:TSSOP-16_4.4x5mm_P0.65mm, F.Cu at (155.5, 108.0)
- added U9: ADS112C04, Package_SO:TSSOP-16_4.4x5mm_P0.65mm, F.Cu at (154.2, 118.2)
- D12, D13, D14: value SK44BL -> BAT54SW; footprint Diode_SMD:D_SMB -> Package_TO_SOT_SMD:SOT-323_SC-70
- J3: footprint Connector_Molex:Molex_Micro-Fit_3.0_43650-0415_1x04_P3.00mm_Vertical -> Connector_Molex:Molex_Micro-Fit_3.0_43650-0515_1x05_P3.00mm_Vertical
- R26: value 100Ω -> 3.3kΩ
- R27, R29: value 100kΩ -> 680
- R28, R30: value 100Ω -> 680
- R31: value 100kΩ -> 10kΩ
- R33: value 10kΩ -> 100kΩ
- R37: value 100kΩ -> 3.3kΩ
- U5: value TPS78450QDBVRQ1 -> TPS7A2050PDBVR
- U6: value ESP32-S3-WROOM-1 -> ESP32-S3-WROOM-1U; footprint RF_Module:ESP32-S3-WROOM-1 -> RF_Module:ESP32-S3-WROOM-1U
- moved R37 93.0 mm to (156.5, 114.2), turned to 0 degrees
- moved R27 92.6 mm to (166.4, 113.9), turned to 90 degrees
- moved D12 90.3 mm to (161.7, 114.0), turned to 180 degrees
- moved R29 89.2 mm to (171.2, 113.9), turned to 90 degrees
- moved R28 88.2 mm to (168.0, 113.9), turned to 90 degrees
- moved R36 87.2 mm to (159.1, 69.5), turned to 0 degrees
- moved R33 86.8 mm to (159.1, 71.1)
- moved Q7 86.1 mm to (158.8, 66.5)
- moved R26 84.8 mm to (153.1, 111.8), turned to 180 degrees
- moved R30 83.1 mm to (169.6, 113.9), turned to 90 degrees
- moved D13 79.0 mm to (161.7, 108.8), turned to 180 degrees
- moved H4 78.7 mm to (172.8, 138.2)
- moved H3 78.1 mm to (116.4, 138.5)
- moved G*** 78.0 mm to (156.4, 111.4)
- moved D14 74.3 mm to (161.7, 111.4), turned to 180 degrees
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Connections:
- net ACTUATOR_1_CTL renamed ACT1_CTL
- net FAN_1_PWM renamed FAN1_PWM
- net FAN_1_TACH renamed FAN1_TACH
- D12 pad 1: +24V -> GND
- D12 pad 2: Net-(D12-A) -> +5V
- D13 pad 1: +24V -> GND
- D13 pad 2: Net-(D13-A) -> +5V
- D14 pad 1: +24V -> GND
- D14 pad 2: Net-(D14-A) -> +5V
- R26 pad 1: ACTUATOR_2_CTL -> +3.3V
- R26 pad 2: Net-(Q3-G) -> DRDY2
- R27 pad 1: ACTUATOR_2_CTL -> /ADC 2/SIG3
- R27 pad 2: GND -> /ADC 2/AIN3
- R28 pad 1: ACTUATOR_3_CTL -> HEAT2_CURR
- R28 pad 2: Net-(Q4-G) -> /ADC 2/AIN2
- R29 pad 1: ACTUATOR_3_CTL -> IGN_CURR
- R29 pad 2: GND -> /ADC 2/AIN1
- R30 pad 1: ACTUATOR_4_CTL -> HEAT1_CURR
- R30 pad 2: Net-(Q5-G) -> /ADC 2/AIN0
- R31 pad 1: ACTUATOR_4_CTL -> +3.3V
- R31 pad 2: GND -> Net-(U8-RESET)
- R33 pad 1: FAN_2_TACH -> ACT2_CTL
- R33 pad 2: +3.3V -> GND
- R36 pad 1: Net-(Q7-G) -> ACT2_CTL
- R36 pad 2: FAN_2_PWM -> Net-(Q7-G)
- R37 pad 1: FAN_2_PWM -> +3.3V
- R37 pad 2: GND -> DRDY3
- R4 pad 1: LOAD_CELL+ -> IGN_RESP
- R5 pad 1: LOAD_CELL- -> IGN_RESN
- R6 pad 1: /ADC 1/SIG1 -> LOAD_CELL+
- R7 pad 1: /ADC 1/SIG0 -> LOAD_CELL-
- U2 pad 4: 5.17V_PG -> unconnected-(U2-PG-Pad4)
- U3 pad 4: 12V_PG -> unconnected-(U3-PG-Pad4)
- U6 pad 10: ACTUATOR_2_CTL -> ACT2_CTL
- U6 pad 17: unconnected-(U6-IO9-Pad17) -> DRDY3
- U6 pad 18: unconnected-(U6-IO10-Pad18) -> DRDY4
- U6 pad 19: unconnected-(U6-IO11-Pad19) -> IGN_PRIME_CTL
- U6 pad 20: unconnected-(U6-IO12-Pad20) -> IGN_RUN_CTL
- U6 pad 21: unconnected-(U6-IO13-Pad21) -> SAFE24_CTL
- U6 pad 22: 5.17V_PG -> HEAT1_PWM
- U6 pad 23: 12V_PG -> HEAT1_ESTOP
- U6 pad 24: unconnected-(U6-IO47-Pad24) -> HEAT2_PWM
- U6 pad 25: unconnected-(U6-IO48-Pad25) -> HEAT2_ESTOP
- U6 pad 31: unconnected-(U6-IO38-Pad31) -> /ESP32 Breakout/WIFI_IND
- U6 pad 34: FAN_2_TACH -> FAN2_TACH
- U6 pad 35: FAN_2_PWM -> FAN2_PWM
- U6 pad 38: unconnected-(U6-IO2-Pad38) -> FAN3_TACH
- U6 pad 39: /ESP32 Breakout/WIFI_IND -> FAN3_PWM
- U6 pad 4: unconnected-(U6-IO4-Pad4) -> DRDY2
- U6 pad 6: I2C_SDA -> I2C_SCL
- U6 pad 7: I2C_SCL -> I2C_SDA
- U6 pad 8: ACTUATOR_4_CTL -> ACT4_CTL
- U6 pad 9: ACTUATOR_3_CTL -> ACT3_CTL
Routing:
- net +5V: track 58.5 -> 283.9 mm, vias 6 -> 27
- net +24V: track 32.9 -> 119.3 mm
- net SAFE24_CTL: track 0.00 -> 66.6 mm, vias 0 -> 1
- net IGN_RUN_CTL: track 0.00 -> 62.8 mm, vias 0 -> 1
- net HEAT2_CURR: track 0.00 -> 62.0 mm, vias 0 -> 2
- net IGN_PRIME_CTL: track 0.00 -> 59.8 mm, vias 0 -> 1
- net HEAT1_PWM: track 0.00 -> 55.0 mm, vias 0 -> 1
- net HEAT2_PWM: track 0.00 -> 54.2 mm, vias 0 -> 1
- net HEAT2_ESTOP: track 0.00 -> 53.7 mm, vias 0 -> 1
- net HEAT1_ESTOP: track 0.00 -> 53.5 mm, vias 0 -> 1
- net GND: track 97.0 -> 142.8 mm, vias 98 -> 135
- net I2C_SDA: track 16.0 -> 59.9 mm
- net DRDY3: track 0.00 -> 43.5 mm, vias 0 -> 2
- net I2C_SCL: track 14.7 -> 57.1 mm, vias 0 -> 4
- net 5.17V_PG: track 42.4 -> 0.00 mm, vias 2 -> 0
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- added copper zone on B.Cu, net GND
Other:
- board size 65 x 65 mm -> 65 x 95 mm
- board text added: "5V + - GND SH"
- board text added: "5V 24V PRIME RUN SAFE24 GND GND RESN RESP CURR"
- board text added: "FAN3"
- board text added: "HEATER1_DRIVER"
- board text added: "HEATER1_TH"
- board text added: "HEATER2_DRIVER"
- board text added: "HEATER2_TH"
- board text added: "IGNITOR_DRIVER"
- board text added: "PWM ESTOP CURR GND 5V 24V"
- board text added: "TH1 TH2 TH3 TH4 GND GND GND GND"
- board text removed: "5V + - GND"
- board text removed: "Footprint does not match for DRC as overhanging silkscreen lines were removed"
- board text removed: "SIG0"
- board text removed: "SIG1"

Commit message: updates for manufacturing
Parts:
- J3: value Conn_01x04 -> Conn_01x05
- R1, R19, R26, R37, R59: value 3.3kΩ -> 3.3k
- R12, R25, R33, R35, R48, R54, R57, R65: value 100kΩ -> 100k
- R13, R15: value 100kΩ -> 100k 0.1%
- R14: value 24kΩ -> 24k 0.1%
- R16: value 9.09kΩ -> 9.09k 0.1%
- R17: value 39kΩ -> 39k
- R18: value 1.2kΩ -> 1.2k
- R2, R21, R3: value 1kΩ -> 1k
- R20, R31, R32, R46, R52, R56, R64, R8, R9: value 10kΩ -> 10k
- R22, R23: value 5.1kΩ -> 5.1k
- R24, R34, R36, R47, R53, R58, R66: value 100Ω -> 100
- R38, R39, R40, R41, R42, R43, R44, R45: value 10k -> 10k 0.1%
- moved G*** 46.6 mm to (150.6, 65.2)
- moved H3 1.13 mm to (117.2, 137.7)
- moved H4 0.78 mm to (172.2, 137.7)
- moved J14 0.30 mm to (130.5, 128.4)
- moved J17 0.30 mm to (130.5, 139.6)
