File: gse_control_node/power_regulation.kicad_sch (KiCad schematic)
At the start: 56 parts, among them J4 Conn_02x01, Q1 DMP6023LE-13, U2 LMR33630BDDA, U3 LMR33630BDDA, U4 TPS78533QKVURQ1, U5 TPS78450QDBVRQ1, U7 LM66200

Commit message: finish control board routing
Parts:
- removed C15: 100uF, Capacitor_SMD:CP_Elec_10x10, symbol Device:C_Polarized_Small_US
- removed R10, R11: 100kΩ, Resistor_SMD:R_0603_1608Metric, symbol Device:R_Small_US
- added C55: 100uF, Capacitor_THT:CP_Radial_D8.0mm_P5.00mm, symbol Device:C_Polarized_Small_US
- U5: value TPS78450QDBVRQ1 -> TPS7A2050PDBVR; LCSC C2877783 -> C2864504
Connections:
- net +24V: now also C55.1
- net GND: now also C55.2
- net 12_POWER_GOOD: no longer names the net of U3.4 (PG)
- net 5.17_POWER_GOOD: no longer names the net of U2.4 (PG)
- no-connect marks 1 -> 3

Commit message: updates for manufacturing
Parts:
- D5, D6, F1, J4, L1, L2, Q1, U4: now in the parts list
- R12: value 100kΩ -> 100k
- R13, R15: value 100kΩ -> 100k 0.1%
- R14: value 24kΩ -> 24k 0.1%
- R16: value 9.09kΩ -> 9.09k 0.1%
- R17: value 39kΩ -> 39k
- R18: value 1.2kΩ -> 1.2k
- R19: value 3.3kΩ -> 3.3k
- R9: value 10kΩ -> 10k
Changed lines of the file:
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@@
 			)
 		)
-		(property "Value" "100kΩ"
-			(at 80.01 167.894 0)
+		(property "Value" "100k 0.1%"
+			(at 79.248 162.052 0)
 			(show_name no)
 			(do_not_autoplace no)
@@
 			)
 		)
-		(property "Value" "100kΩ"
+		(property "Value" "100k"
 			(at 74.93 44.4499 0)
 			(show_name no)
@@
 		(body_style 1)
 		(exclude_from_sim no)
-		(in_bom no)
+		(in_bom yes)
 		(on_board yes)
-		(in_pos_files no)
+		(in_pos_files yes)
 		(dnp no)
 		(property "Reference" "D5"
@@
 		(body_style 1)
 		(exclude_from_sim no)
-		(in_bom no)
+		(in_bom yes)
 		(on_board yes)
-		(in_pos_files no)
+		(in_pos_files yes)
 		(dnp no)
 		(property "Reference" "F1"
@@
 			)
 		)
-		(property "Value" "9.09kΩ"
+		(property "Value" "9.09k 0.1%"
 			(at 80.264 173.99 0)
 			(show_name no)
@@
 		(body_style 1)
 		(exclude_from_sim no)
-		(in_bom no)
+		(in_bom yes)
 		(on_board yes)
-		(in_pos_files no)
+		(in_pos_files yes)
 		(dnp no)
 		(property "Reference" "L2"
@@
 		(body_style 1)
 		(exclude_from_sim no)
-		(in_bom no)
+		(in_bom yes)
 		(on_board yes)
-		(in_pos_files no)
+		(in_pos_files yes)
 		(dnp no)
 		(property "Reference" "Q1"
@@
 			)
 		)
-		(property "Value" "24kΩ"
+		(property "Value" "24k 0.1%"
 			(at 80.264 109.22 0)
 			(show_name no)
@@
 		(body_style 1)
 		(exclude_from_sim no)
-		(in_bom no)
+		(in_bom yes)
 		(on_board yes)
-		(in_pos_files no)
+		(in_pos_files yes)
 		(dnp no)
 		(property "Reference" "U4"
@@
 		(body_style 1)
 		(exclude_from_sim no)
-		(in_bom no)
+		(in_bom yes)
 		(on_board yes)
-		(in_pos_files no)
+		(in_pos_files yes)
 		(dnp no)
 		(fields_autoplaced yes)
@@
 			)
 		)
-		(property "Value" "3.3kΩ"
+		(property "Value" "3.3k"
 			(at 262.382 101.854 0)
 			(show_name no)
@@
 			)
 		)
-		(property "Value" "39kΩ"
+		(property "Value" "39k"
 			(at 110.236 45.72 0)
 			(show_name no)
@@
 			)
 		)
-		(property "Value" "10kΩ"
+		(property "Value" "10k"
 			(at 58.42 53.3399 0)
 			(show_name no)
@@
 			)
 		)
-		(property "Value" "100kΩ"
-			(at 80.01 103.124 0)
+		(property "Value" "100k 0.1%"
+			(at 79.502 97.536 0)
 			(show_name no)
 			(do_not_autoplace no)
@@
 		(body_style 1)
 		(exclude_from_sim no)
-		(in_bom no)
+		(in_bom yes)
 		(on_board yes)
-		(in_pos_files no)
+		(in_pos_files yes)
 		(dnp no)
 		(property "Reference" "D6"
@@
 		(in_bom yes)
 		(on_board yes)
-		(in_pos_files no)
+		(in_pos_files yes)
 		(dnp no)
 		(property "Reference" "C55"
@@
 		(body_style 1)
 		(exclude_from_sim no)
-		(in_bom no)
+		(in_bom yes)
 		(on_board yes)
-		(in_pos_files no)
+		(in_pos_files yes)
 		(dnp no)
 		(property "Reference" "L1"
@@
 			)
 		)
-		(property "Value" "1.2kΩ"
+		(property "Value" "1.2k"
 			(at 196.342 104.394 0)
 			(show_name no)
