File: gse_control_node/power_regulation.kicad_sch (KiCad schematic)
At the start: 56 parts, among them J4 Conn_02x01, Q1 DMP6023LE-13, U2 LMR33630BDDA, U3 LMR33630BDDA, U4 TPS78533QKVURQ1, U5 TPS78450QDBVRQ1, U7 LM66200

Commit message: Heater/ignitor control (#2)
* update project to kicad v10

* remove thermistors from board

* rename project to be more descriptive

* fix load cell connector

* switch to on-board esp32s3

* fix fan header footprint

* update buck converter components and add reverse polarity protection

* do some pcb routing

* finish pcb routing

* remove unneccesary component fields

* add all lcsc part numbers

* add readme

* add thermal reliefs on bottom power planes

* give more clearance for load cell connector from edge of board

* fix 5.17V buck switch node net name

* switch to esp32-s3-wroom-1

* update some routing and put ground pour on top layer to avoid warping

* update silkscreen

* update all capacitors to jlcpcb basic components

* add a 12v testpoint

* update resistors to jlcpcb basic components

* fix copper pour priorities

* move up ads112c04 capacitors further from pins for easier handsoldering

* remove some extended components from bom (to be handsoldered)

* update screw terminal footprint

* add tachometer pullup and pwm low side fet for fans

* organize hierarchical sheet page numbers

* add heater connectors

* add heater power regulation for fet switching

* seperate board directories and finish heater driver routing

* add relay to heater board for estop and do some ignitor board routing

* finish ignitor board routing

* finish control board routing

* updates for manufacturing

* remove leftover files

* improve silkscreening on ignitor board and add connector for keyswitch

* make gitignore ignore production dir recursively
Parts:
- removed C15: 100uF, Capacitor_SMD:CP_Elec_10x10, symbol Device:C_Polarized_Small_US
- removed R10, R11: 100kΩ, Resistor_SMD:R_0603_1608Metric, symbol Device:R_Small_US
- added C55: 100uF, Capacitor_THT:CP_Radial_D8.0mm_P5.00mm, symbol Device:C_Polarized_Small_US
- D5, D6, F1, J4, L1, L2, Q1, U4: now in the parts list
- R12: value 100kΩ -> 100k
- R13, R15: value 100kΩ -> 100k 0.1%
- R14: value 24kΩ -> 24k 0.1%
- R16: value 9.09kΩ -> 9.09k 0.1%
- R17: value 39kΩ -> 39k
- R18: value 1.2kΩ -> 1.2k
- R19: value 3.3kΩ -> 3.3k
- R9: value 10kΩ -> 10k
- U5: value TPS78450QDBVRQ1 -> TPS7A2050PDBVR; LCSC C2877783 -> C2864504
Connections:
- net +24V: now also C55.1
- net GND: now also C55.2
- net 12_POWER_GOOD: no longer names the net of U3.4 (PG)
- net 5.17_POWER_GOOD: no longer names the net of U2.4 (PG)
- no-connect marks 1 -> 3
