File: ignitor_driver/ignitor_driver.kicad_pcb (KiCad board)
At the start: 2 copper layers, 70 x 65 mm, 51 parts, among them J1 Conn_02x05_Counter_Clockwise, J4 Conn_02x01, K1 G5LE-1 DC24, K2 G5LE-1 DC24, K3 G5LE-1 DC24, Q1 PMOS, Q2 BSS138, Q3 BSS138, Q4 BSS138, U1 LM4040DBZ-2.5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

Commit message: finish ignitor board routing
Parts:
- added J2: 24V_IN, Library:AMT0440007DB0000G, F.Cu at (164.5, 116.0)
- added J3: GND_IN, Library:AMT0440007DB0000G, F.Cu at (108.5, 116.0)
- moved H2 12.5 mm to (119.0, 117.0)
- moved H3 12.5 mm to (154.0, 117.0)
- moved J4 4.85 mm to (106.5, 107.3), turned to 180 degrees
- moved J1 4.05 mm to (130.5, 115.2)
- moved C12 3.66 mm to (152.3, 92.8)
- moved C6 0.51 mm to (147.2, 91.5)
- moved C7 0.51 mm to (147.2, 93.7)
- moved C11 0.45 mm to (158.3, 92.3)
Connections:
- J4 pad 1: Net-(J4-Pin_1) -> GND_ISO
- J4 pad 2: GND_ISO -> Net-(J4-Pin_2)
- U6 pad 3: Net-(J4-Pin_1) -> Net-(J4-Pin_2)
- U6 pad 4: Net-(J4-Pin_1) -> Net-(J4-Pin_2)
Routing:
- net /PRIME_CTL_CONN: track 4.04 -> 146.6 mm
- net /RUN_CTL_CONN: track 20.8 -> 109.7 mm
- net /SAFE24_CTL_CONN: track 4.04 -> 89.8 mm
- net /24V_CONN: track 77.6 -> 159.4 mm
- net /GND_CONN: track 137.4 -> 195.4 mm
- net GND_ISO: track 182.5 -> 239.5 mm, vias 7 -> 8
- net +24V_ISO: track 67.6 -> 104.5 mm
- net /5V_CONN: track 69.8 -> 61.7 mm
- net /CURR_CONN: track 64.3 -> 57.1 mm
- net Net-(J4-Pin_1): track 3.86 -> 0.00 mm
- net Net-(J4-Pin_2): track 0.00 -> 3.61 mm
- net /RESN_CONN: track 9.99 -> 12.7 mm
- net /RESP_CONN: track 10.0 -> 11.0 mm
- net /R_SENSE: track 14.9 -> 14.0 mm
- net Net-(U5-DCDC_OUT): track 10.5 -> 9.88 mm
- added copper zone on B.Cu, net GND_ISO
- added copper zone on F.Cu, net GND_ISO
- added copper zone on B.Cu, net Net-(J2-Pin_1)
- added copper zone on F.Cu, net Net-(J2-Pin_1)
- added copper zone on F.Cu, net Net-(J4-Pin_2)
- removed copper zone on F.Cu, net Net-(J4-Pin_1)

Commit message: updates for manufacturing
Parts:
- R3: value 10k -> 10k 0.1%
- R5: value 30k -> 30k 0.1%
- R7: footprint Resistor_SMD:R_0805_2012Metric_Pad1.20x1.40mm_HandSolder -> Resistor_SMD:R_0603_1608Metric_Pad0.98x0.95mm_HandSolder
- U6: value ACS713ELCTR-20A-T -> ACS724xLCTR-30AU
Routing:
- net GND_ISO: track 239.5 -> 234.4 mm
