File: ignitor_driver/ignitor_driver.kicad_pcb (KiCad board)
At the start: 2 copper layers, 70 x 65 mm, 53 parts, among them J1 Conn_02x05_Counter_Clockwise, J2 24V_IN, J3 GND_IN, J4 Conn_02x01, K1 G5LE-1 DC24, K2 G5LE-1 DC24, K3 G5LE-1 DC24, Q1 PMOS, Q2 BSS138, Q3 BSS138, Q4 BSS138, U1 LM4040DBZ-2.5, U2 LM4040DBZ-2.5, U3 TLV333IDBVR, U4 OPA990IDBVR, U5 AMC3330, U6 ACS724xLCTR-30AU

Commit message: improve silkscreening on ignitor board and add connector for keyswitch
Parts:
- added J5: Lockout, Connector_Molex:Molex_Mini-Fit_Jr_5566-02A_2x01_P4.20mm_Vertical, F.Cu at (167.3, 105.5)
- J4: value Conn_02x01 -> Ignitor
Connections:
- F1 pad 1: Net-(J2-Pin_1) -> Net-(J5-Pin_2)
Routing:
- net Net-(J5-Pin_2): track 0.00 -> 13.2 mm
Other:
- board text added: "24V_ISO"
- board text added: "CURR RESP RESN GND GND SAFE24 RUN PRIME 24V 5V"
- board text added: "GND_ISO"
